Commit message: [WIP] First pass combining vehicle and arm together
- Combined vehicle and arm URDFs into one within `base.xacro`
- Still need to do more extensive testing showing where
  the arm is located relative to the vehicle
- `upload.launch` does not work

File: seabotix_alpha_description/urdf/base.xacro (robot description, xacro)
@@ -59,4 +59,536 @@
         </collision>
       </link>
+      <!-- robot name="OSU vLBV300 Volturnus" -->
+      <xacro:property name="pi" value="3.1515926535897931" />
+      <xacro:property name="deg2rad" value="${pi/180}" />
+      <!-- Without trig, angles are a pain in the arse. Beam angle 30 -->
+      <xacro:property name="dvl_beam_angle" value="${30/180*pi}" />
+      <xacro:property name="dvl_pitch" value="0.361367" />
+      <xacro:property name="dvl_yaw" value="0.387597" />
+      <material name="green">
+        <color rgba="0.5 0.9 0.3 1"/>
+      </material>
+      <material name="black">
+        <color rgba="0 0 0 1"/>
+      </material>
+      <material name="red">
+        <color rgba="1 0 0 1"/>
+      </material>
+      <material name="blue">
+        <color rgba="0.2 0.4 0.6 1" />
+      </material>
+      <material name="grey">
+        <color rgba=".3 .3 .3 1"/>
+      </material>
+      <material name="orange">
+        <color rgba="1 .4 0 1" />
+      </material>
+      <link name="vehicle_base_link">
+        <visual>
+          <geometry>
+            <box size="0.5 0.45 0.15"/>
+          </geometry>
+          <material name="green"/>
+        </visual>
+      </link>
+      <link name="front_bumper">
+        <visual>
+          <geometry>
+            <cylinder length="0.45" radius="0.075"/>
+          </geometry>
+          <material name="green"/>
+        </visual>
+      </link>
+      <joint name="fbump_link" type="fixed">
+        <parent link="vehicle_base_link"/>
+        <child link="front_bumper"/>
+        <origin rpy="${pi/2} 0 0" xyz="0.25 0 0"/>
+      </joint>
+      <link name="rear_bumper">
+        <visual>
+          <geometry>
+            <cylinder length="0.45" radius="0.075"/>
+          </geometry>
+          <material name="green"/>
+        </visual>
+      </link>
+      <joint name="rbump_link" type="fixed">
+        <parent link="vehicle_base_link"/>
+        <child link="rear_bumper"/>
+        <origin rpy="${pi/2} 0 0" xyz="-0.25 0 0"/>
+      </joint>
+      <link name="l_arrow">
+        <visual>
+          <geometry>
+            <box size="0.05 0.318 0.01"/>
+          </geometry>
+          <material name="black"/>
+        </visual>
+      </link>
+      <joint name="l_arrow_link" type="fixed">
+        <parent link="vehicle_base_link"/>
+        <child link="l_arrow"/>
+        <origin rpy="0 0 ${pi/4}" xyz="0.05 0.095 0.075"/>
+      </joint>
+      <link name="r_arrow">
+        <visual>
+          <geometry>
+            <box size="0.05 0.318 0.01"/>
+          </geometry>
+          <material name="black"/>
+        </visual>
+      </link>
+      <joint name="r_arrow_link" type="fixed">
+        <parent link="vehicle_base_link"/>
+        <child link="r_arrow"/>
+        <origin rpy="0 0 ${-pi/4}" xyz="0.05 -0.095 0.075"/>
+      </joint>
+      <link name="sf_fan">
+        <visual>
+          <geometry>
+            <cylinder length="0.04" radius="0.06"/>
+          </geometry>
+          <material name="blue"/>
+        </visual>
+      </link>
+      <joint name="base_to_sf_fan" type="fixed">
+        <parent link="vehicle_base_link"/>
+        <child link="sf_fan"/>
+        <origin rpy="0 ${pi/2} 0.785" xyz="0.22 -0.12 -0.14"/>
+      </joint>
+      <link name="sf_thruster">
+        <visual>
+          <geometry>
+            <cylinder length="0.1" radius="0.02"/>
+          </geometry>
+          <material name="black"/>
+        </visual>
+      </link>
+      <joint name="sf_fan_thruster_joint" type="fixed">
+        <parent link="sf_fan"/>
+        <child link="sf_thruster"/>
+        <origin xyz="0 0 -0.06"/>
+      </joint>
+      <link name="pf_fan">
+        <visual>
+          <geometry>
+            <cylinder length="0.04" radius="0.06"/>
+          </geometry>
+          <material name="blue"/>
+        </visual>
+      </link>
+      <joint name="base_to_pf_fan" type="fixed">
+        <parent link="vehicle_base_link"/>
+        <child link="pf_fan"/>
+        <origin rpy="0 ${pi/2} -0.785" xyz="0.22 0.12 -0.14"/>
+      </joint>
+      <link name="pf_thruster">
+        <visual>
+          <geometry>
+            <cylinder length="0.1" radius="0.02"/>
+          </geometry>
+          <material name="black"/>
+        </visual>
+      </link>
+      <joint name="pf_fan_thruster_joint" type="fixed">
+        <parent link="pf_fan"/>
+        <child link="pf_thruster"/>
+        <origin xyz="0 0 -0.06"/>
+      </joint>
+      <link name="sa_fan">
+        <visual>
+          <geometry>
+            <cylinder length="0.04" radius="0.06"/>
+          </geometry>
+          <material name="blue"/>
+        </visual>
+      </link>
+      <joint name="base_to_sa_fan" type="fixed">
+        <parent link="vehicle_base_link"/>
+        <child link="sa_fan"/>
+        <origin rpy="0 ${-pi/2} -0.785" xyz="-0.22 -0.12 -0.14"/>
+      </joint>
+      <link name="sa_thruster">
+        <visual>
+          <geometry>
+            <cylinder length="0.1" radius="0.02"/>
+          </geometry>
+          <material name="black"/>
+        </visual>
+      </link>
+      <joint name="sa_fan_thruster_joint" type="fixed">
+        <parent link="sa_fan"/>
+        <child link="sa_thruster"/>
+        <origin xyz="0 0 -0.06"/>
+      </joint>
+      <link name="pa_fan">
+        <visual>
+          <geometry>
+            <cylinder length="0.04" radius="0.06"/>
+          </geometry>
+          <material name="blue"/>
+        </visual>
+      </link>
+      <joint name="base_to_pa_fan" type="fixed">
+        <parent link="vehicle_base_link"/>
+        <child link="pa_fan"/>
+        <origin rpy="0 -${pi/2} 0.785" xyz="-0.22 0.12 -0.14"/>
+      </joint>
+      <link name="pa_thruster">
+        <visual>
+          <geometry>
+            <cylinder length="0.1" radius="0.02"/>
+          </geometry>
+          <material name="black"/>
+        </visual>
+      </link>
+      <joint name="pa_fan_thruster_joint" type="fixed">
+        <parent link="pa_fan"/>
+        <child link="pa_thruster"/>
+        <origin xyz="0 0 -0.06"/>
+      </joint>
+      <link name="seabotix_bottle">
+        <visual>
+          <geometry>
+            <cylinder length="0.26" radius="0.05"/>
+          </geometry>
+          <material name="black"/>
+        </visual>
+      </link>
+      <joint name="sbottle_link" type="fixed">
+        <parent link="vehicle_base_link"/>
+        <child link="seabotix_bottle"/>
+        <origin rpy="0 ${pi/2} 0" xyz="-0.05 0 -0.18"/>
+      </joint>
+      <link name="greensea">
+        <visual>
+          <geometry>
+            <cylinder length="0.2" radius="0.04"/>
+          </geometry>
+          <origin rpy="0 ${pi/2} 0"/>
+          <material name="grey"/>
+        </visual>
+      </link>
+      <joint name="gbottle_link" type="fixed">
+        <parent link="greensea"/>
+        <child link="vehicle_base_link"/>
+        <origin rpy="-${pi} 0 0" xyz="0 0 -0.27"/>
+      </joint>
+      <link name="dvl">
+        <visual>
+          <geometry>
+            <cylinder length="0.25" radius="0.06"/>
+          </geometry>
+          <material name="grey"/>
+          <origin rpy="0 ${pi/2} 0" xyz="-0.125 0 0"/>
+        </visual>
+      </link>
+      <joint name="dvl_link" type="fixed">
+        <parent link="vehicle_base_link"/>
+        <child link="dvl"/>
+        <origin rpy="0 0 ${pi}" xyz="-0.23 -0.1 -0.29"/>
+      </joint>
+      <link name="dvl_head">
+        <visual>
+          <geometry>
+            <sphere radius="0.06"/>
+          </geometry>
+          <material name="orange"/>
+        </visual>
+      </link>
+      <joint name="dvl_head_link" type="fixed">
+        <parent link="dvl"/>
+        <child link="dvl_head"/>
+        <origin rpy="0 0 ${-45*deg2rad}" xyz="0 0 0"/>
+      </joint>
+      <link name="dvl_altitude"/>
+      <joint name="dvl_altitude_link" type="fixed">
+        <parent link="dvl_head"/>
+        <child link="dvl_altitude"/>
+        <origin rpy="0 ${pi/2} 0" xyz="0 0 0"/>
+      </joint>
+      <link name="dvl_beam1">
+        <visual>
+          <geometry>
+            <cylinder length="0.07" radius="0.015"/>
+          </geometry>
+          <origin rpy="0 ${pi/2} 0" xyz="0.035 0 0"/>
+          <material name="blue"/>
+        </visual>
+      </link>
+      <joint name="dvl_beam1_link" type="fixed">
+        <parent link="dvl_head"/>
+        <child link="dvl_beam1"/>
+        <origin rpy="0 ${pi/2-dvl_beam_angle} ${pi/2}" xyz="0 0 0"/>
+      </joint>
+      <link name="dvl_beam2">
+        <visual>
+          <geometry>
+            <cylinder length="0.07" radius="0.015"/>
+          </geometry>
+          <origin rpy="0 ${pi/2} 0" xyz="0.035 0 0"/>
+          <material name="blue"/>
+        </visual>
+      </link>
+      <joint name="dvl_beam2_link" type="fixed">
+        <parent link="dvl_head"/>
+        <child link="dvl_beam2"/>
+        <origin rpy="0 ${pi/2-dvl_beam_angle} -${pi/2}" xyz="0 0 0"/>
+      </joint>
+      <link name="dvl_beam3">
+        <visual>
+          <geometry>
+            <cylinder length="0.07" radius="0.015"/>
+          </geometry>
+          <origin rpy="0 ${pi/2} 0" xyz="0.035 0 0"/>
+          <material name="blue"/>
+        </visual>
+      </link>
+      <joint name="dvl_beam3_link" type="fixed">
+        <parent link="dvl_head"/>
+        <child link="dvl_beam3"/>
+        <origin rpy="0 ${pi/2-dvl_beam_angle} 0" xyz="0 0 0"/>
+      </joint>
+      <link name="dvl_beam4">
+        <visual>
+          <geometry>
+            <cylinder length="0.07" radius="0.015"/>
+          </geometry>
+          <origin rpy="0 ${pi/2} 0" xyz="0.035 0 0"/>
+          <material name="blue"/>
+        </visual>
+      </link>
+      <joint name="dvl_beam4_link" type="fixed">
+        <parent link="dvl_head"/>
+        <child link="dvl_beam4"/>
+        <origin rpy="0 ${pi/2-dvl_beam_angle} ${pi}" xyz="0 0 0"/>
+      </joint>
+      <link name="sonar">
+        <visual>
+          <geometry>
+            <box size="0.22 0.13 0.1"/>
+          </geometry>
+          <material name="orange"/>
+        </visual>
+      </link>
+      <joint name="sonar_link" type="fixed">
+        <parent link="vehicle_base_link"/>
+        <child link="sonar"/>
+        <origin xyz="0.1 0.12 -0.28"/>
+      </joint>
+      <link name="gripper_pole">
+        <visual>
+          <geometry>
+            <cylinder length="0.38" radius="0.015"/>
+          </geometry>
+          <origin rpy="0 ${pi/2} 0" xyz="0.19 0 0"/>
+          <material name="black"/>
+        </visual>
+      </link>
+      <joint name="gripper_pole_link" type="fixed">
+        <parent link="vehicle_base_link"/>
+        <child link="gripper_pole"/>
+        <origin rpy="0 0.1 0.3" xyz="0.15 -0.15 -0.2"/>
+      </joint>
+<material name="black">
+  <color rgba="0 0 0 1"/>
+</material>
+  <link name="arm_base_link">
+    <visual>
+      <geometry>
+	<mesh filename="package://reach_system_one_support/meshes/reach5mini/visual/Base.stl" />
+      </geometry>
+      <origin rpy="0 0 0" xyz="0 0 0"/>
+      <material name="black"/>
+    </visual>
+    <collision>
+      <geometry>
+        <cylinder length="0.150" radius="0.020"/>
+      </geometry>
+      <origin rpy="0 1.57075 0" xyz="-0.075 0 0"/>
+    </collision>
+    <inertial>
+      <mass value="0.341"/>
+      <origin xyz="-0.075 -0.006 -0.003"/>
+      <inertia ixx="0.000099" ixy="0.000139" ixz="0.000115" iyy="0.002920" iyz="0.000003" izz="0.002934"/>
+    </inertial>
+  </link>
+  <link name="shoulder_link">
+    <visual>
+      <geometry>
+        <mesh filename="package://reach_system_one_support/meshes/reach5mini/visual/ShoulderJoint.stl" />
+      </geometry>
+      <material name="black"/>
+      <origin rpy="0 0 -1.57075" xyz="0 0 0"/>
+    </visual>
+    <collision>
+      <geometry>
+        <cylinder length="0.066" radius="0.020"/>
+      </geometry>
+      <origin rpy="0 0 0" xyz="0 0 0.010"/>
+    </collision>
+    <inertial>
+      <mass value="0.194"/>
+      <origin xyz="0.005 -0.001 0.016"/>
+      <inertia ixx="0.000189" ixy="0.000005" ixz="0.000054" iyy="0.000213" iyz="0.000003" izz="0.000067"/>
+    </inertial>
+  </link>
+  <link name="upper_arm_link">
+    <visual>
+      <geometry>
+        <mesh filename="package://reach_system_one_support/meshes/reach5mini/visual/UpperArm.stl" />
+      </geometry>
+      <origin rpy="0 -1.57075 -0.2655555" xyz="0 0 -0.075"/>
+      <material name="black"/>
+    </visual>
+    <collision>
+      <geometry>
+        <cylinder length="0.1445" radius="0.020"/>
+      </geometry>
+      <origin rpy="0 1.57075 -0.27075" xyz="0.075 0 0"/>
+    </collision>
+    <collision>
+      <geometry>
+        <cylinder length="0.040" radius="0.020"/>
+      </geometry>
+      <origin rpy="0 0 0" xyz="0 0 0"/>
+    </collision>
+    <inertial>
+      <mass value="0.429"/>
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