Commit message: WIP Simulate UVMS system
- Vehicle + Arm in the simulator
- Still running into issues where thrusters are getting Nan.
- This is becaus Gazebo is reporting the angular portion of the state as nan

TO DO:
- Debug why Gazebo pose_gt is reporting Nan angular pose

File: seabotix_alpha_description/urdf/actuators_backup.xacro (robot description, xacro)
@@ -8,29 +8,42 @@
           aware that Gazebo does not use the SNAME convention per default.
     -->
+  <xacro:property name="prop_mesh_file" value="file://$(find seabotix_alpha_description)/meshes/prop_scaled.dae"/>
+  <!-- Thruster joint and link snippet -->
+  <xacro:macro name="thruster_macro"
+    params="namespace thruster_id *origin">
+    <xacro:thruster_module_first_order_basic_fcn_macro
+      namespace="${namespace}"
+      thruster_id="${thruster_id}"
+      mesh_filename="${prop_mesh_file}"
+      dyn_time_constant="0.05"
+      rotor_constant="0.00031">
+      <xacro:insert_block name="origin"/>
+    </xacro:thruster_module_first_order_basic_fcn_macro>
+  </xacro:macro>
     <!-- Correspond to PA (Port Aft) fan in urdf -->
-    <!-- <xacro:thruster_macro robot_namespace="${namespace}" thruster_id="0">
+    <xacro:thruster_macro robot_namespace="${namespace}" thruster_id="0">
         <origin xyz="-0.22 -0.12 ${-0.27+0.14}" rpy="${-pi} {-pi/2} 0.785" />
-    </xacro:thruster_macro> -->
+    </xacro:thruster_macro>
     <!-- Correspond to PF (Port Forward) fan in urdf -->
-    <!-- <xacro:thruster_macro robot_namespace="${namespace}" thruster_id="1">
+    <xacro:thruster_macro robot_namespace="${namespace}" thruster_id="1">
         <origin xyz="0.22 -0.12 ${-0.27+0.14}" rpy="${-pi} {pi/2} -0.785" />
-    </xacro:thruster_macro> -->
+    </xacro:thruster_macro>
     <!-- Correspond to SA (Starboard Aft) fan in urdf -->
-    <!-- <xacro:thruster_macro robot_namespace="${namespace}" thruster_id="2">
+    <xacro:thruster_macro robot_namespace="${namespace}" thruster_id="2">
         <origin xyz="-0.22 0.12 ${-0.27+0.14}" rpy="${-pi} {-pi/2} -0.785" />
-    </xacro:thruster_macro> -->
+    </xacro:thruster_macro>
     <!-- Correspond to SF (Starboard Forward) fan in urdf -->
-    <!-- <xacro:thruster_macro robot_namespace="${namespace}" thruster_id="3">
+    <xacro:thruster_macro robot_namespace="${namespace}" thruster_id="3">
         <origin xyz="0.22 0.12 ${-0.27+0.14}" rpy="${-pi} {pi/2} 0.785" />
-    </xacro:thruster_macro> -->
+    </xacro:thruster_macro>
 <!-- Vertical fans estimated -->
     <!-- Correspond to VP (Vertical Port) fan (not in urdf) -->
-    <!-- <xacro:thruster_macro robot_namespace="${namespace}" thruster_id="4">
+    <xacro:thruster_macro robot_namespace="${namespace}" thruster_id="4">
         <origin xyz="0.22 -0.10 0" rpy="0 0 0" />
-    </xacro:thruster_macro> -->
+    </xacro:thruster_macro>
         <!-- Correspond to SF (Vertical Starboard) fan (not in urdf) -->
-    <!-- <xacro:thruster_macro robot_namespace="${namespace}" thruster_id="5">
+    <xacro:thruster_macro robot_namespace="${namespace}" thruster_id="5">
         <origin xyz="0.22 0.10 0 " rpy="0 0 0" />
-    </xacro:thruster_macro> -->
+    </xacro:thruster_macro>
     <!-- Instantiate fins, if necessary -->
     <!-- <xacro:fin_macro namespace="${namespace}" fin_id="0">
@@ -46,17 +59,4 @@
       <origin xyz="0 0 0" rpy="0 0 0" />
     </xacro:fin_macro> -->
-  <xacro:property name="prop_mesh_file" value="file://$(find seabotix_alpha_description)/meshes/prop_scaled.dae"/>
-  <!-- Thruster joint and link snippet -->
-  <xacro:macro name="thruster_macro"
-    params="namespace thruster_id *origin">
-    <xacro:thruster_module_first_order_basic_fcn_macro
-      namespace="${namespace}"
-      thruster_id="${thruster_id}"
-      mesh_filename="${prop_mesh_file}"
-      dyn_time_constant="0.05"
-      rotor_constant="0.00031">
-      <xacro:insert_block name="origin"/>
-    </xacro:thruster_module_first_order_basic_fcn_macro>
-  </xacro:macro>
   <!-- Rexrov thrusters - change these later -->
   <!-- <xacro:thruster_macro namespace="${namespace}" thruster_id="0">
@@ -84,36 +84,3 @@
     <origin xyz="0.412125 -0.505415 0.129" rpy="${0*d2r} ${0*d2r} ${-135*d2r}"/>
   </xacro:thruster_macro> -->
-    <!-- Correspond to PA (Port Aft) fan in urdf -->
-    <xacro:thruster_macro namespace="${namespace}" thruster_id="0">
-        <origin xyz="-0.22 -0.12 ${-0.27+0.14}" rpy="${-pi} ${-pi/2} 0.785" />
-    </xacro:thruster_macro>
-    <!-- Correspond to PF (Port Forward) fan in urdf -->
-    <xacro:thruster_macro namespace="${namespace}" thruster_id="1">
-        <origin xyz="0.22 -0.12 ${-0.27+0.14}" rpy="${-pi} ${pi/2} -0.785" />
-    </xacro:thruster_macro>
-    <!-- Correspond to SA (Starboard Aft) fan in urdf -->
-    <xacro:thruster_macro namespace="${namespace}" thruster_id="2">
-        <origin xyz="-0.22 0.12 ${-0.27+0.14}" rpy="${-pi} ${-pi/2} -0.785" />
-    </xacro:thruster_macro>
-    <!-- Correspond to SF (Starboard Forward) fan in urdf -->
-    <xacro:thruster_macro namespace="${namespace}" thruster_id="3">
-        <origin xyz="0.22 0.12 ${-0.27+0.14}" rpy="${-pi} ${pi/2} 0.785" />
-    </xacro:thruster_macro>
-<!-- Vertical fans estimated -->
-    <!-- Correspond to VP (Vertical Port) fan (not in urdf) -->
-    <xacro:thruster_macro namespace="${namespace}" thruster_id="4">
-        <origin xyz="0.22 -0.10 0" rpy="0 0 0" />
-    </xacro:thruster_macro>
-        <!-- Correspond to SF (Vertical Starboard) fan (not in urdf) -->
-    <xacro:thruster_macro namespace="${namespace}" thruster_id="5">
-        <origin xyz="0.22 0.10 0 " rpy="0 0 0" />
-    </xacro:thruster_macro>
-        <!-- Dummy thruster to match number of thrusters in rexrov -->
-    <xacro:thruster_macro namespace="${namespace}" thruster_id="6">
-        <origin xyz="0.0 0.0 0.0 " rpy="0 0 0" />
-    </xacro:thruster_macro>
-        <!-- Dummy thruster to match number of thrusters in rexrov -->
-    <xacro:thruster_macro namespace="${namespace}" thruster_id="7">
-        <origin xyz="0.0 0.0 0.0 " rpy="0 0 0" />
-    </xacro:thruster_macro>
 </robot>

File: seabotix_alpha_description/urdf/seabotix.gazebo.xacro (robot description, xacro)
@@ -9,5 +9,5 @@
     <xacro:property name="seabotix_alpha_width"  value="0"/>
     <xacro:property name="seabotix_alpha_height" value="0"/>
-    <xacro:macro name="seabotix_alpha_hydro_model" params="namespace">
+    <xacro:macro name="seabotix_hydro_model" params="namespace">
       <!-- List of hydrodynamic models this robot's links -->
       <link name="${namespace}/base_link">
@@ -36,11 +36,12 @@
         <hydrodynamic_model>
           <type>fossen</type>
+          <!-- Added mass: see p.28 in Berg2012 -->
           <added_mass>
-            0 0 0 0 0 0
-            0 0 0 0 0 0
-            0 0 0 0 0 0
-            0 0 0 0 0 0
-            0 0 0 0 0 0
-            0 0 0 0 0 0
+             1 0 0 0 0 0
+             0 1 0 0 0 0
+             0 0 1 0 0 0
+             0 0 0 1 0 0
+             0 0 0 0 1 0
+             0 0 0 0 0 1
           </added_mass>
           <!--
@@ -48,6 +49,7 @@
             or a full matrix (36 coefficients), like the added-mass coefficients above
           -->
+          <!-- Linear damping: see p.31 in Berg2012 -->
           <linear_damping>
-            0 0 0 0 0 0
+            1 1 1 1 1 1
           </linear_damping>
           <!--
@@ -64,6 +66,7 @@
             or a full matrix (36 coefficients), like the added-mass coefficients above
           -->
+          <!-- Non-linear damping: see p.30 in Berg2012 -->
           <quadratic_damping>
-            0 0 0 0 0 0
+              0 0 0 0 0 0
           </quadratic_damping>
           <!--

File: seabotix_alpha_description/urdf/seabotix_base_components.xacro (robot description, xacro)
@@ -1,38 +1,59 @@
-<?xml version="1.0"?>
-<robot xmlns:xacro="http://www.ros.org/wiki/xacro">
-  <!-- Loading some constants -->
-  <xacro:include filename="$(find uuv_descriptions)/urdf/common.urdf.xacro"/>
-  <!-- Loading file with sensor macros -->
-  <xacro:include filename="$(find uuv_sensor_ros_plugins)/urdf/sensor_snippets.xacro"/>
-  <!-- Loading the UUV simulator ROS plugin macros -->
-  <xacro:include filename="$(find uuv_gazebo_ros_plugins)/urdf/snippets.xacro"/>
-  <!-- Loading vehicle's specific macros -->
-  <xacro:include filename="$(find seabotix_alpha_description)/urdf/snippets.xacro"/>
-  <!--
-    Vehicle's parameters (remember to enter the model parameters below)
-  -->
-  <xacro:property name="mass" value="0"/>
-  <!-- Center of gravity -->
-  <xacro:property name="cog" value="0 0 0"/>
-  <!-- Fluid density -->
-  <xacro:property name="rho" value="1028"/>
-  <!--
-    Visual mesh file for the vehicle, usually in DAE (Collada) format. Be sure to store the
-    mesh with the origin of the mesh on the same position of the center of mass, otherwise
-    the mesh pose will have to be corrected below in the <visual> block.
-    Open the meshes for the RexROV vehicle in Blender to see an example on the mesh placement.
-  -->
-  <!-- <xacro:property name="visual_mesh_file" value="file://$(find seabotix_alpha_description)/meshes/vehicle.dae"/> -->
-  <!-- Collision geometry mesh, usually in STL format (it is recommended to keep
-  this geometry as simple as possible to improve the performance the physics engine
-  regarding the computation of collision forces) -->
-  <!-- <xacro:property name="collision_mesh_file" value="file://$(find seabotix_alpha_description)/meshes/vehicle.stl"/> -->
-  <!-- We do not have different visual and collision files, as we define them directly in the URDF
-       using primitive shapes.
-  -->
-  <!-- Vehicle macro -->
-  <xacro:macro name="seabotix_alpha_base" params="namespace *gazebo">
+    <link name="base_link">
+        <inertial>
+        <mass value="${mass}" />
+        <origin xyz="${cog}" rpy="0 0 0"/>
+        <inertia ixx="0" ixy="0" ixz="0"
+                iyy="0" iyz="0"
+                izz="0" />
+        </inertial>
+    </link>
+    <link name="world_link_x">
+        <inertial>
+        <mass value="0" />
+        <origin xyz="0" rpy="0 0 0"/>
+        <inertia ixx="0" ixy="0" ixz="0"
+                iyy="0" iyz="0"
+                izz="0" />
+        </inertial>
+    </link>
+    <link name="world_link_y">
+        <inertial>
+        <mass value="0" />
+        <origin xyz="0" rpy="0 0 0"/>
+        <inertia ixx="0" ixy="0" ixz="0"
+                iyy="0" iyz="0"
+                izz="0" />
+        </inertial>
+    </link>
+    <link name="world_link_z">
+        <inertial>
+        <mass value="0" />
+        <origin xyz="0" rpy="0 0 0"/>
+        <inertia ixx="0" ixy="0" ixz="0"
+                iyy="0" iyz="0"
+                izz="0" />
+        </inertial>
+    </link>
+    <link name="world_link_roll">
+        <inertial>
+        <mass value="0" />
+        <origin xyz="0" rpy="0 0 0"/>
+        <inertia ixx="0" ixy="0" ixz="0"
+                iyy="0" iyz="0"
+                izz="0" />
+        </inertial>
+    </link>
+    <link name="world_link_pitch">
+        <inertial>
+        <mass value="0" />
+        <origin xyz="0" rpy="0 0 0"/>
+        <inertia ixx="0" ixy="0" ixz="0"
+                iyy="0" iyz="0"
+                izz="0" />
+        </inertial>
+    </link>
       <!-- Rigid body description of the base link -->
-      <link name="${namespace}/base_link">
+      <!-- <link name="${namespace}/base_link"> -->
+      <link name="world_link_yaw">
         <!--
           Be careful to setup the coefficients for the inertial tensor,
@@ -40,14 +61,16 @@
         -->
         <inertial>
-          <mass value="${mass}" />
-          <origin xyz="${cog}" rpy="0 0 0"/>
+          <mass value="0" />
+          <origin xyz="0" rpy="0 0 0"/>
           <inertia ixx="0" ixy="0" ixz="0"
                    iyy="0" iyz="0"
                    izz="0" />
         </inertial>
-        <visual>
+        <!-- <visual>
           <origin xyz="0 0 0" rpy="0 0 0"/>
-          <geometry>
-            <mesh filename="${visual_mesh_file}" scale="1 1 1" />
+          <geometry> -->
+            <!-- <mesh filename="${visual_mesh_file}" scale="1 1 1" />  -->
+            <!-- <box size="1 1 1" />
+            <color rgb="blue" />
           </geometry>
         </visual>
@@ -55,7 +78,7 @@
           <origin xyz="0 0 0" rpy="0 0 0"/>
           <geometry>
-            <mesh filename="${collision_mesh_file}" scale="1 1 1" />
-          </geometry>
-        </collision>
+            <box size="1 1 1" />
+          </geometry>
+        </collision> -->
       </link>
       <!-- robot name="OSU vLBV300 Volturnus" -->
@@ -66,20 +89,20 @@
       <xacro:property name="dvl_pitch" value="0.361367" />
       <xacro:property name="dvl_yaw" value="0.387597" />
-      <material name="green">
+      <material name="green_v">
         <color rgba="0.5 0.9 0.3 1"/>
       </material>
-      <material name="black">
+      <material name="black_v">
         <color rgba="0 0 0 1"/>
       </material>
-      <material name="red">
+      <material name="red_v">
         <color rgba="1 0 0 1"/>
       </material>
-      <material name="blue">
+      <material name="blue_v">
         <color rgba="0.2 0.4 0.6 1" />
       </material>
-      <material name="grey">
+      <material name="grey_v">
         <color rgba=".3 .3 .3 1"/>
       </material>
-      <material name="orange">
+      <material name="orange_v">
         <color rgba="1 .4 0 1" />
       </material>
@@ -89,5 +112,5 @@
             <box size="0.5 0.45 0.15"/>
           </geometry>
-          <material name="green"/>
+          <material name="green_v"/>
         </visual>
       </link>
@@ -97,5 +120,5 @@
             <cylinder length="0.45" radius="0.075"/>
           </geometry>
-          <material name="green"/>
+          <material name="green_v"/>
         </visual>
       </link>
@@ -110,5 +133,5 @@
             <cylinder length="0.45" radius="0.075"/>
           </geometry>
-          <material name="green"/>
+          <material name="green_v"/>
         </visual>
       </link>
@@ -123,5 +146,5 @@
             <box size="0.05 0.318 0.01"/>
           </geometry>
-          <material name="black"/>
+          <material name="black_v"/>
         </visual>
       </link>
@@ -136,5 +159,5 @@
             <box size="0.05 0.318 0.01"/>
           </geometry>
-          <material name="black"/>
+          <material name="black_v"/>
         </visual>
       </link>
@@ -149,5 +172,5 @@
             <cylinder length="0.04" radius="0.06"/>
           </geometry>
-          <material name="blue"/>
+          <material name="blue_v"/>
         </visual>
       </link>
@@ -162,5 +185,5 @@
             <cylinder length="0.1" radius="0.02"/>
           </geometry>
-          <material name="black"/>
+          <material name="black_v"/>
         </visual>
       </link>
@@ -175,5 +198,5 @@
             <cylinder length="0.04" radius="0.06"/>
           </geometry>
-          <material name="blue"/>
+          <material name="blue_v"/>
         </visual>
       </link>
@@ -188,5 +211,5 @@
             <cylinder length="0.1" radius="0.02"/>
           </geometry>
-          <material name="black"/>
+          <material name="black_v"/>
         </visual>
       </link>
@@ -201,5 +224,5 @@
             <cylinder length="0.04" radius="0.06"/>
           </geometry>
-          <material name="blue"/>
+          <material name="blue_v"/>
         </visual>
       </link>
@@ -214,5 +237,5 @@
             <cylinder length="0.1" radius="0.02"/>
           </geometry>
-          <material name="black"/>
+          <material name="black_v"/>
         </visual>
       </link>
@@ -227,5 +250,5 @@
             <cylinder length="0.04" radius="0.06"/>
           </geometry>
-          <material name="blue"/>
+          <material name="blue_v"/>
         </visual>
       </link>
@@ -240,5 +263,5 @@
             <cylinder length="0.1" radius="0.02"/>
           </geometry>
-          <material name="black"/>
+          <material name="black_v"/>
         </visual>
       </link>
@@ -253,5 +276,5 @@
             <cylinder length="0.26" radius="0.05"/>
           </geometry>
-          <material name="black"/>
+          <material name="black_v"/>
         </visual>
       </link>
@@ -261,4 +284,5 @@
         <origin rpy="0 ${pi/2} 0" xyz="-0.05 0 -0.18"/>
       </joint>
+<!--
       <link name="greensea">
         <visual>
@@ -267,5 +291,5 @@
           </geometry>
           <origin rpy="0 ${pi/2} 0"/>
-          <material name="grey"/>
+          <material name="grey_v"/>
         </visual>
       </link>
@@ -274,5 +298,5 @@
         <child link="vehicle_base_link"/>
         <origin rpy="-${pi} 0 0" xyz="0 0 -0.27"/>
-      </joint>
+      </joint> -->
       <link name="dvl">
         <visual>
@@ -280,5 +304,5 @@
             <cylinder length="0.25" radius="0.06"/>
           </geometry>
-          <material name="grey"/>
+          <material name="grey_v"/>
           <origin rpy="0 ${pi/2} 0" xyz="-0.125 0 0"/>
         </visual>
@@ -294,5 +318,5 @@
             <sphere radius="0.06"/>
           </geometry>
-          <material name="orange"/>
+          <material name="orange_v"/>
         </visual>
       </link>
@@ -314,5 +338,5 @@
           </geometry>
           <origin rpy="0 ${pi/2} 0" xyz="0.035 0 0"/>
-          <material name="blue"/>
+          <material name="blue_v"/>
         </visual>
       </link>
@@ -328,5 +352,5 @@
           </geometry>
           <origin rpy="0 ${pi/2} 0" xyz="0.035 0 0"/>
-          <material name="blue"/>
+          <material name="blue_v"/>
         </visual>
       </link>
@@ -342,5 +366,5 @@
           </geometry>
           <origin rpy="0 ${pi/2} 0" xyz="0.035 0 0"/>
-          <material name="blue"/>
+          <material name="blue_v"/>
         </visual>
       </link>
@@ -356,5 +380,5 @@
           </geometry>
           <origin rpy="0 ${pi/2} 0" xyz="0.035 0 0"/>
-          <material name="blue"/>
+          <material name="blue_v"/>
         </visual>
       </link>
@@ -369,5 +393,5 @@
             <box size="0.22 0.13 0.1"/>
           </geometry>
-          <material name="orange"/>
+          <material name="orange_v"/>
         </visual>
       </link>
@@ -383,5 +407,5 @@
           </geometry>
           <origin rpy="0 ${pi/2} 0" xyz="0.19 0 0"/>
-          <material name="black"/>
+          <material name="black_v"/>
         </visual>
       </link>
@@ -391,213 +415,51 @@
         <origin rpy="0 0.1 0.3" xyz="0.15 -0.15 -0.2"/>
       </joint>
-<material name="black">
-  <color rgba="0 0 0 1"/>
-</material>
-  <link name="arm_base_link">
-    <visual>
-      <geometry>
-	<mesh filename="package://reach_system_one_support/meshes/reach5mini/visual/Base.stl" />
-      </geometry>
-      <origin rpy="0 0 0" xyz="0 0 0"/>
-      <material name="black"/>
-    </visual>
-    <collision>
-      <geometry>
-        <cylinder length="0.150" radius="0.020"/>
-      </geometry>
-      <origin rpy="0 1.57075 0" xyz="-0.075 0 0"/>
-    </collision>
-    <inertial>
-      <mass value="0.341"/>
-      <origin xyz="-0.075 -0.006 -0.003"/>
-      <inertia ixx="0.000099" ixy="0.000139" ixz="0.000115" iyy="0.002920" iyz="0.000003" izz="0.002934"/>
-    </inertial>
-  </link>
-  <link name="shoulder_link">
-    <visual>
-      <geometry>
-        <mesh filename="package://reach_system_one_support/meshes/reach5mini/visual/ShoulderJoint.stl" />
-      </geometry>
-      <material name="black"/>
-      <origin rpy="0 0 -1.57075" xyz="0 0 0"/>
-    </visual>
-    <collision>
-      <geometry>
-        <cylinder length="0.066" radius="0.020"/>
-      </geometry>
-      <origin rpy="0 0 0" xyz="0 0 0.010"/>
-    </collision>
-    <inertial>
-      <mass value="0.194"/>
-      <origin xyz="0.005 -0.001 0.016"/>
-      <inertia ixx="0.000189" ixy="0.000005" ixz="0.000054" iyy="0.000213" iyz="0.000003" izz="0.000067"/>
-    </inertial>
-  </link>
-  <link name="upper_arm_link">
-    <visual>
-      <geometry>
-        <mesh filename="package://reach_system_one_support/meshes/reach5mini/visual/UpperArm.stl" />
-      </geometry>
-      <origin rpy="0 -1.57075 -0.2655555" xyz="0 0 -0.075"/>
-      <material name="black"/>
-    </visual>
-    <collision>
-      <geometry>
-        <cylinder length="0.1445" radius="0.020"/>
-      </geometry>
-      <origin rpy="0 1.57075 -0.27075" xyz="0.075 0 0"/>
-    </collision>
-    <collision>
-      <geometry>
-        <cylinder length="0.040" radius="0.020"/>
-      </geometry>
-      <origin rpy="0 0 0" xyz="0 0 0"/>
-    </collision>
-    <inertial>
-      <mass value="0.429"/>
-      <origin xyz="0.073 0.0 0.0"/>
-      <inertia ixx="0.000087" ixy="-0.000076" ixz="-0.000010" iyy="0.003190" iyz="0.000000" izz="0.003213"/>
-    </inertial>
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