Commit message: Base Mesh Conversion
- Retrying adapting seabotix vehicle from RexRov Base
- Replace rexrov base with seabotix vehicle

File: seabotix_alpha_description/urdf/rexrov_oberon7.xacro (robot description, xacro)
@@ -12,12 +12,12 @@
      limitations under the License.
 -->
-<robot name="seabotix" xmlns:xacro="http://www.ros.org/wiki/xacro" >
+<robot name="rexrov" xmlns:xacro="http://www.ros.org/wiki/xacro" >
   <xacro:arg name="debug" default="0"/>
-  <xacro:arg name="namespace" default="seabotix"/>
+  <xacro:arg name="namespace" default="rexrov"/>
   <xacro:arg name="inertial_reference_frame" default="world"/>
   <!-- Include the ROV macro file -->
-  <xacro:include filename="$(find seabotix_alpha_description)/urdf/seabotix_base.xacro"/>
-  <xacro:include filename="$(find seabotix_alpha_description)/urdf/seabotix.gazebo.xacro"/>
-  <xacro:include filename="$(find seabotix_alpha_description)/urdf/alpha_default.xacro" />
+  <xacro:include filename="$(find seabotix_alpha_description)/urdf/rexrov_base.xacro"/>
+  <xacro:include filename="$(find seabotix_alpha_description)/urdf/rexrov.gazebo.xacro"/>
+  <xacro:include filename="$(find uuv_dave)/urdf/oberon7_default.xacro" />
   <xacro:uuv_forward_looking_sonar
       namespace="${namespace}"
@@ -57,5 +57,5 @@
 -->
   <!-- Create the ROV -->
-  <xacro:seabotix_base
+  <xacro:rexrov_base
     namespace="$(arg namespace)"
     inertial_reference_frame="$(arg inertial_reference_frame)">
@@ -68,13 +68,12 @@
         <debug>$(arg debug)</debug>
         <!-- Adding the hydrodynamic and hydrostatic parameters for the vehicle-->
-        <xacro:seabotix_hydro_model namespace="$(arg namespace)"/>
-        <xacro:alpha_hydro_model namespace="alpha"/>
+        <xacro:rexrov_hydro_model namespace="$(arg namespace)"/>
+        <xacro:oberon7_hydro_model namespace="oberon7"/>
       </plugin>
     </gazebo>
-  </xacro:seabotix_base>
-  <xacro:alpha namespace="alpha" parent="$(arg namespace)/base_link">
-  <!-- TODO Update this origin relative to seabotix base -->
-    <origin rpy="0 0 0" xyz="0.45 0 0"/> <!--TODO: Update this-->
-  </xacro:alpha>
+  </xacro:rexrov_base>
+  <xacro:oberon7 namespace="oberon7" parent="$(arg namespace)/base_link">
+    <origin xyz="1.3 -0.5 -0.615" rpy="0 0 0"/>
+  </xacro:oberon7>
   <gazebo>
       <plugin name="gazebo_ros_control" filename="libgazebo_ros_control.so">

File: seabotix_alpha_description/urdf/rexrov_sensors.xacro (robot description, xacro)
@@ -1,16 +1,16 @@
 <?xml version="1.0"?>
+<!-- Copyright (c) 2016 The UUV Simulator Authors.
+     All rights reserved.
+     Licensed under the Apache License, Version 2.0 (the "License");
+     you may not use this file except in compliance with the License.
+     You may obtain a copy of the License at
+       http://www.apache.org/licenses/LICENSE-2.0
+     Unless required by applicable law or agreed to in writing, software
+     distributed under the License is distributed on an "AS IS" BASIS,
+     WITHOUT WARRANTIES OR CONDITIONS OF ANY KIND, either express or implied.
+     See the License for the specific language governing permissions and
+     limitations under the License.
+-->
 <robot xmlns:xacro="http://www.ros.org/wiki/xacro">
-  <!--
-    Some examples of sensors that can be added to the vehicle frame.
-    Set the origin of the sensor frames correctly for your application
-    Look into the sensor macros in the package uuv_sensor_ros_plugins/urdf for
-    more examples or add you own custom sensor units.
-  -->
-  <!-- Mount a Pose 3D sensor. -->
-  <!-- <xacro:default_pose_3d namespace="${namespace}" parent_link="${namespace}/base_link" /> -->
-  <!-- Forward-looking sonar sensor -->
-  <!-- <xacro:forward_multibeam_p900 namespace="${namespace}" parent_link="${namespace}/base_link">
-    <origin xyz="0 0 0" rpy="0 0 0"/>
-  </xacro:forward_multibeam_p900> -->
   <!-- DVL  -->
   <xacro:default_dvl_macro
@@ -20,14 +20,14 @@
     <origin xyz="-1.4 0 -0.312" rpy="0 ${0.5*pi} 0"/>
   </xacro:default_dvl_macro>
- <!-- Magnetometer  -->
+  <!-- Magnetometer  -->
   <xacro:default_magnetometer namespace="${namespace}" parent_link="${namespace}/base_link"/>
   <!-- RPT  -->
   <xacro:default_rpt namespace="${namespace}" parent_link="${namespace}/base_link">
-    <origin xyz="0 0 0" rpy="0 0 0"/>
+    <origin xyz="-1.32 0 0.8" rpy="0 0 0"/>
   </xacro:default_rpt>
   <!-- Pressure  -->
-  <xacro:default_pressure namespace="${namespace}" parent_link="${namespace}/base_link">
-    <origin xyz="0 0 0" rpy="0 0 0"/>
-  </xacro:default_pressure>
+  <xacro:default_pressure_macro namespace="${namespace}" parent_link="${namespace}/base_link">
+    <origin xyz="-1.32 0.5 0.85" rpy="0 0 0"/>
+  </xacro:default_pressure_macro>
   <!-- IMU  -->
   <xacro:default_imu_macro
@@ -37,18 +37,13 @@
     <origin xyz="0 0 0" rpy="0 0 0"/>
   </xacro:default_imu_macro>
-  <!-- Mount a camera  -->
-  <!-- <xacro:default_camera namespace="${namespace}" parent_link="${namespace}/base_link" suffix="">
-    <origin xyz="0 0 0" rpy="0 0 0"/>
-  </xacro:default_camera> -->
-<!-- Rexrov systems -->
   <!-- Mount a camera -->
   <xacro:default_camera namespace="${namespace}" parent_link="${namespace}/base_link" suffix="">
-    <origin xyz="0.3 0 0.4" rpy="0 0.6 0"/>
+    <origin xyz="1.15 0 0.4" rpy="0 0.6 0"/>
   </xacro:default_camera>
   <xacro:default_camera namespace="${namespace}" parent_link="${namespace}/base_link" suffix="right">
-    <origin xyz="0.3 -0.1 0.4" rpy="0 0.6 0.4"/>
+    <origin xyz="1.15 -0.63 0.4" rpy="0 0.6 0.4"/>
   </xacro:default_camera>
   <xacro:default_camera namespace="${namespace}" parent_link="${namespace}/base_link" suffix="left">
-    <origin xyz="0.3 0.1 0.4" rpy="0 0.6 -0.4"/>
+    <origin xyz="1.15 0.63 0.4" rpy="0 0.6 -0.4"/>
   </xacro:default_camera>
   <!-- Mount a GPS. -->
