Commit message: Moving rexrov/oberon7 dependencies to this repo

File: seabotix_alpha_description/urdf/oberon7_default.xacro (robot description, xacro)
@@ -12,11 +12,11 @@
      limitations under the License.
 -->
-<robot name="alpha" xmlns:xacro="http://www.ros.org/wiki/xacro">
+<robot name="oberon7" xmlns:xacro="http://www.ros.org/wiki/xacro">
   <!-- Import serial arm -->
-  <xacro:include filename="$(find seabotix_alpha_description)/urdf/alpha_arm.xacro" />
+  <xacro:include filename="$(find seabotix_alpha_description)/urdf/serial_arm.xacro" />
   <!-- Import Gazebo specific macros -->
-  <xacro:include filename="$(find seabotix_alpha_description)/urdf/alpha_arm.gazebo.xacro" />
-  <xacro:macro name="alpha" params="namespace parent *origin">
-    <xacro:alpha_arm namespace="${namespace}"/>
+  <xacro:include filename="$(find seabotix_alpha_description)/urdf/serial_arm.gazebo.xacro" />
+  <xacro:macro name="oberon7" params="namespace parent *origin">
+    <xacro:oberon7_serial_arm namespace="${namespace}"/>
     <joint name="${namespace}/anchor" type="revolute">
       <parent link="${parent}"/>

File: seabotix_alpha_description/urdf/rexrov_oberon7.xacro (robot description, xacro)
@@ -19,5 +19,5 @@
   <xacro:include filename="$(find seabotix_alpha_description)/urdf/rexrov_base.xacro"/>
   <xacro:include filename="$(find seabotix_alpha_description)/urdf/rexrov.gazebo.xacro"/>
-  <xacro:include filename="$(find uuv_dave)/urdf/oberon7_default.xacro" />
+  <xacro:include filename="$(find seabotix_alpha_description)/urdf/oberon7_default.xacro" />
   <xacro:uuv_forward_looking_sonar
       namespace="${namespace}"
