Commit message: Added Alpha arm without any controller/actuator
- Simply placed the alpha arm URDF into the model
- oberon7 arm is still there
- Alpha arm has no controller at the moment

File: seabotix_alpha_description/urdf/alpha_default.xacro (robot description, xacro)
@@ -21,5 +21,5 @@
     <joint name="${namespace}/anchor" type="revolute">
       <parent link="${parent}"/>
-      <child link="${namespace}/base"/>
+      <child link="${namespace}/base_link"/>
       <xacro:insert_block name="origin"/>
       <axis xyz="0 1 0"/>

File: seabotix_alpha_description/urdf/rexrov_oberon7.xacro (robot description, xacro)
@@ -20,4 +20,5 @@
   <xacro:include filename="$(find seabotix_alpha_description)/urdf/rexrov.gazebo.xacro"/>
   <xacro:include filename="$(find seabotix_alpha_description)/urdf/oberon7_default.xacro" />
+  <xacro:include filename="$(find seabotix_alpha_description)/urdf/alpha_default.xacro" />
   <xacro:uuv_forward_looking_sonar
       namespace="${namespace}"
@@ -70,4 +71,5 @@
         <xacro:rexrov_hydro_model namespace="$(arg namespace)"/>
         <xacro:oberon7_hydro_model namespace="oberon7"/>
+        <!-- <xacro:alpha_hydro_model namespace="alpha"/> -->
       </plugin>
     </gazebo>
@@ -76,4 +78,7 @@
     <origin xyz="1.3 -0.5 -0.615" rpy="0 0 0"/>
   </xacro:oberon7>
+  <xacro:alpha namespace="alpha" parent="$(arg namespace)/base_link">
+    <origin xyz="1.3 0.5 -0.615" rpy="0 0 0"/>
+  </xacro:alpha>
   <gazebo>
       <plugin name="gazebo_ros_control" filename="libgazebo_ros_control.so">
