Commit message: Changed arm inertia parameters
- Used cylinder and rectangular prism approximations
  for inertias of links in alpha arm

File: seabotix_alpha_description/urdf/alpha_arm.gazebo.xacro (robot description, xacro)
@@ -3,8 +3,4 @@
   <xacro:include filename="$(find seabotix_alpha_description)/urdf/alpha_arm_ft_sensor.xacro" />
   <xacro:macro name="alpha_gazebo_macro" params="namespace">
-    <gazebo reference="${namespace}/base">
-      <selfCollide>false</selfCollide>
-      <maxContacts>1</maxContacts>
-    </gazebo>
     <gazebo reference="${namespace}/base_link">
       <selfCollide>false</selfCollide>
@@ -64,9 +60,9 @@
     <link name="${namespace}/base_link">
       <volume>${pi*(0.020**2)*0.150}</volume>
-      <!-- <box>
-        <width>${base_width}</width>
-        <length>${base_length}</length>
-        <height>${base_height}</height>
-      </box> -->
+      <box>
+        <width>${0.020*2}</width>
+        <height>${0.020*2}</height>
+        <length>${0.150}</length>
+      </box>
       <hydrodynamic_model>
         <type>cylinder</type>
@@ -76,9 +72,9 @@
     <link name="${namespace}/shoulder_link">
       <volume>${pi*(0.020**2)*0.066}</volume>
-      <!-- <box>
-        <width>${shoulder_link_width}</width>
-        <length>${shoulder_link_length}</length>
-        <height>${shoulder_link_height}</height>
-      </box> -->
+      <box>
+        <width>${0.020*2}</width>
+        <height>${0.020*2}</height>
+        <length>${0.066}</length>
+      </box>
       <hydrodynamic_model>
         <type>cylinder</type>
@@ -88,9 +84,9 @@
     <link name="${namespace}/upper_arm_link">
       <volume>${pi*(0.020**2)*0.1445}</volume>
-      <!-- <box>
-        <width>${upper_arm_width}</width>
-        <length>${upper_arm_length}</length>
-        <height>${upper_arm_height}</height>
-      </box> -->
+      <box>
+        <width>${0.020*2}</width>
+        <height>${0.020*2}</height>
+        <length>${0.1445}</length>
+      </box>
       <hydrodynamic_model>
         <type>cylinder</type>
@@ -100,9 +96,9 @@
     <link name="${namespace}/forearm_link">
       <volume>${pi*(0.020**2)*0.040}</volume>
-      <!-- <box>
-        <width>${elbow_link_width}</width>
-        <length>${elbow_link_length}</length>
-        <height>${elbow_link_height}</height>
-      </box> -->
+      <box>
+        <width>${0.020*2}</width>
+        <height>${0.020*2}</height>
+        <length>${0.040}</length>
+      </box>
       <hydrodynamic_model>
         <type>cylinder</type>
@@ -112,9 +108,9 @@
     <link name="${namespace}/wrist_link">
       <volume>${pi*(0.020**2)*0.140}</volume>
-      <!-- <box>
-        <width>${wrist_width}</width>
-        <length>${wrist_length}</length>
-        <height>${wrist_height}</height>
-      </box> -->
+      <box>
+        <width>${0.020*2}</width>
+        <height>${0.020*2}</height>
+        <length>${0.140}</length>
+      </box>
       <hydrodynamic_model>
         <type>cylinder</type>

File: seabotix_alpha_description/urdf/alpha_arm.xacro (robot description, xacro)
@@ -22,5 +22,5 @@
         </joint>
         <actuator name="${joint}_motor">
-          <hardwareInterface>EffortJointInterface</hardwareInterface>
+          <!-- <hardwareInterface>EffortJointInterface</hardwareInterface> -->
           <mechanicalReduction>1</mechanicalReduction>
         </actuator>
@@ -68,5 +68,8 @@
             <mass value="0.194"/>
             <origin xyz="0.005 -0.001 0.016"/>
-            <inertia ixx="0.000189" ixy="0.000005" ixz="0.000054" iyy="0.000213" iyz="0.000003" izz="0.000067"/>
+            <!-- <inertia ixx="0.000189" ixy="0.000005" ixz="0.000054" iyy="0.000213" iyz="0.000003" izz="0.000067"/> -->
+            <inertia ixx="${(1/12)*0.194*(0.066)**2 + 0.25*0.194*0.020**2}" ixy="0.0" ixz="0.0"
+            iyy="${(1/12)*0.194*(0.066)**2 + 0.25*0.194*0.020**2}" iyz="0.0"
+            izz="${0.5*0.194*0.020**2}"/>
             </inertial>
         </link>
@@ -94,5 +97,9 @@
             <mass value="0.429"/>
             <origin xyz="0.073 0.0 0.0"/>
-            <inertia ixx="0.000087" ixy="-0.000076" ixz="-0.000010" iyy="0.003190" iyz="0.000000" izz="0.003213"/>
+            <!-- <inertia ixx="0.000087" ixy="-0.000076" ixz="-0.000010" iyy="0.003190" iyz="0.000000" izz="0.003213"/>
+            </inertial> -->
+            <inertia ixx="${(1/12)*0.429*(0.040)**2 + 0.25*0.429*0.020**2}" ixy="0.25" ixz="0.0"
+            iyy="${(1/12)*0.429*(0.040)**2 + 0.25*0.429*0.020**2}" iyz="0.0"
+            izz="${0.5*0.429*0.020**2}"/>
             </inertial>
         </link>
@@ -114,5 +121,9 @@
             <mass value="0.115"/>
             <origin xyz="0.017 -0.026 -0.002"/>
-            <inertia ixx="0.000120" ixy="-0.000061" ixz="-0.000001" iyy="0.000062" iyz="0.000000" izz="0.000156"/>
+            <!-- <inertia ixx="0.000120" ixy="-0.000061" ixz="-0.000001" iyy="0.000062" iyz="0.000000" izz="0.000156"/>
+            </inertial> -->
+            <inertia ixx="${(1/12)*0.115*(0.040)**2 + 0.25*0.115*0.020**2}" ixy="0.0" ixz="0.0"
+            iyy="${(1/12)*0.115*(0.040)**2 + 0.25*0.115*0.020**2}" iyz="0.0"
+            izz="${0.5*0.115*0.020**2}"/>
             </inertial>
         </link>
@@ -134,5 +145,9 @@
             <mass value="0.333"/>
             <origin xyz="0.0 0.003 -0.098"/>
-            <inertia ixx="0.003709" ixy="-0.000002" ixz="-0.000004" iyy="0.003734" iyz="0.000000" izz="0.000079"/>
+            <!-- <inertia ixx="0.003709" ixy="-0.000002" ixz="-0.000004" iyy="0.003734" iyz="0.000000" izz="0.000079"/>
+            </inertial> -->
+            <inertia ixx="${(1/12)*0.333*(0.040)**2 + 0.25*0.333*0.140**2}" ixy="0.0" ixz="0.0"
+            iyy="${(1/12)*0.333*(0.040)**2 + 0.25*0.333*0.140**2}" iyz="0.0"
+            izz="${0.5*0.333*0.140**2}"/>
             </inertial>
         </link>
@@ -157,5 +172,8 @@
             <mass value="0.333"/>
             <origin xyz="0.0 0.003 -0.098"/>
-            <inertia ixx="0.003709" ixy="-0.000002" ixz="-0.000004" iyy="0.003734" iyz="0.000000" izz="0.000079"/>
+            <!-- <inertia ixx="0.003709" ixy="-0.000002" ixz="-0.000004" iyy="0.003734" iyz="0.0" izz="0.000079"/> -->
+            <inertia ixx="${1/12*0.333*(0.09**2+0.01**2)}" ixy="0.0" ixz="-0.0"
+            iyy="${1/12*0.333*(0.03**2+0.01**2)}" iyz="0.0"
+            izz="${1/12*0.333*(0.03**2+0.09**2)}"/>
             </inertial>
         </link>
@@ -178,6 +196,9 @@
             <mass value="0.333"/>
             <origin xyz="0.0 0.003 -0.098"/>
-            <inertia ixx="0.003709" ixy="-0.000002" ixz="-0.000004" iyy="0.003734" iyz="0.000000" izz="0.000079"/>
-            </inertial>
+            <!-- <inertia ixx="0.003709" ixy="-0.00002" ixz="-0.00004" iyy="0.003734" iyz="0.0" izz="0.000079"/> -->
+            <inertia ixx="${1/12*0.333*(0.09**2+0.01**2)}" ixy="0.0" ixz="-0.0"
+            iyy="${1/12*0.333*(0.03**2+0.01**2)}" iyz="0.0"
+            izz="${1/12*0.333*(0.03**2+0.09**2)}"/>
+            </inertial>-->
         </link>
         <joint name="${namespace}/joint1" type="revolute">

File: seabotix_alpha_description/urdf/rexrov_oberon7.xacro (robot description, xacro)
@@ -71,5 +71,5 @@
         <xacro:rexrov_hydro_model namespace="$(arg namespace)"/>
         <xacro:oberon7_hydro_model namespace="oberon7"/>
-        <!-- <xacro:alpha_hydro_model namespace="alpha"/> -->
+        <xacro:alpha_hydro_model namespace="alpha"/>
       </plugin>
     </gazebo>
