Commit message: Removed Oberon Arm, Reposition Alpha Arm
- Oberon arm removed from model
- Alpha arm repositioned to a reasonable location.
- Added damping/friction terms to alpha arm joints to try to control stability.
- Alpha arm still jitters.
- Increasing damping too much/changing PID terms can cause the simulation to become
  unstable and the model to fail.

File: seabotix_alpha_description/urdf/alpha_arm.xacro (robot description, xacro)
@@ -49,4 +49,7 @@
             <origin xyz="-0.075 -0.006 -0.003"/>
             <inertia ixx="0.000099" ixy="0.000139" ixz="0.000115" iyy="0.002920" iyz="0.000003" izz="0.002934"/>
+            <!-- <inertia ixx="${(1/12)*0.341*(0.150)**2 + 0.25*0.341*0.020**2}" ixy="0.0" ixz="0.0"
+            iyy="${(1/12)*0.341*(0.150)**2 + 0.25*0.341*0.020**2}" iyz="0.0"
+            izz="${0.5*0.341*0.020**2}"/> -->
             </inertial>
         </link>
@@ -97,6 +100,5 @@
             <mass value="0.429"/>
             <origin xyz="0.073 0.0 0.0"/>
-            <!-- <inertia ixx="0.000087" ixy="-0.000076" ixz="-0.000010" iyy="0.003190" iyz="0.000000" izz="0.003213"/>
-            </inertial> -->
+            <!-- <inertia ixx="0.000087" ixy="-0.000076" ixz="-0.000010" iyy="0.003190" iyz="0.000000" izz="0.003213"/> -->
             <inertia ixx="${(1/12)*0.429*(0.040)**2 + 0.25*0.429*0.020**2}" ixy="0.25" ixz="0.0"
             iyy="${(1/12)*0.429*(0.040)**2 + 0.25*0.429*0.020**2}" iyz="0.0"
@@ -121,6 +123,5 @@
             <mass value="0.115"/>
             <origin xyz="0.017 -0.026 -0.002"/>
-            <!-- <inertia ixx="0.000120" ixy="-0.000061" ixz="-0.000001" iyy="0.000062" iyz="0.000000" izz="0.000156"/>
-            </inertial> -->
+            <!-- <inertia ixx="0.000120" ixy="-0.000061" ixz="-0.000001" iyy="0.000062" iyz="0.000000" izz="0.000156"/> -->
             <inertia ixx="${(1/12)*0.115*(0.040)**2 + 0.25*0.115*0.020**2}" ixy="0.0" ixz="0.0"
             iyy="${(1/12)*0.115*(0.040)**2 + 0.25*0.115*0.020**2}" iyz="0.0"
@@ -145,6 +146,5 @@
             <mass value="0.333"/>
             <origin xyz="0.0 0.003 -0.098"/>
-            <!-- <inertia ixx="0.003709" ixy="-0.000002" ixz="-0.000004" iyy="0.003734" iyz="0.000000" izz="0.000079"/>
-            </inertial> -->
+            <!-- <inertia ixx="0.003709" ixy="-0.000002" ixz="-0.000004" iyy="0.003734" iyz="0.000000" izz="0.000079"/> -->
             <inertia ixx="${(1/12)*0.333*(0.040)**2 + 0.25*0.333*0.140**2}" ixy="0.0" ixz="0.0"
             iyy="${(1/12)*0.333*(0.040)**2 + 0.25*0.333*0.140**2}" iyz="0.0"
@@ -156,24 +156,26 @@
         <link name="${namespace}/jaw1">
             <visual>
-            <geometry>
-                <mesh filename="package://reach_system_one_support/meshes/reach5mini/visual/Jaw1.stl" />
-            </geometry>
-            <origin rpy="0 0 0" xyz="0 0 0"/>
-            <material name="black_arm"/>
-            </visual>
-            <collision>
-            <geometry>
-                <box size="0.03 0.09 0.01"/>
-            </geometry>
-            <origin rpy="0 0 0" xyz="-0.01 -0.045 0"/>
+                <geometry>
+                    <mesh filename="package://reach_system_one_support/meshes/reach5mini/visual/Jaw1.stl" />
+                </geometry>
+                <origin rpy="0 0 0" xyz="0 0 0"/>
+                <material name="black_arm"/>
+            </visual>
+            <collision>
+                <geometry>
+                    <!-- <box size="0.03 0.09 0.01"/> -->
+                    <box size="0.02 0.07 0.01"/>
+                </geometry>
+                <!-- <origin rpy="0 0 0" xyz="-0.01 -0.045 0"/> -->
+                <origin rpy="0 0 0" xyz="-0.02 -0.045 0"/>
             </collision>
             <!-- Made up inertias from wrist -->
             <inertial>
-            <mass value="0.333"/>
-            <origin xyz="0.0 0.003 -0.098"/>
-            <!-- <inertia ixx="0.003709" ixy="-0.000002" ixz="-0.000004" iyy="0.003734" iyz="0.0" izz="0.000079"/> -->
-            <inertia ixx="${1/12*0.333*(0.09**2+0.01**2)}" ixy="0.0" ixz="-0.0"
-            iyy="${1/12*0.333*(0.03**2+0.01**2)}" iyz="0.0"
-            izz="${1/12*0.333*(0.03**2+0.09**2)}"/>
+                <mass value="0.333"/>
+                <origin xyz="0.0 0.003 -0.098"/>
+                <!-- <inertia ixx="0.003709" ixy="-0.000002" ixz="-0.000004" iyy="0.003734" iyz="0.0" izz="0.000079"/> -->
+                <inertia ixx="${1/12*0.333*(0.09**2+0.01**2)}" ixy="0.0" ixz="-0.0"
+                iyy="${1/12*0.333*(0.03**2+0.01**2)}" iyz="0.0"
+                izz="${1/12*0.333*(0.03**2+0.09**2)}"/>
             </inertial>
         </link>
@@ -187,8 +189,10 @@
             </visual>
             <collision>
-            <geometry>
-                <box size="0.03 0.09 0.01"/>
-            </geometry>
-            <origin rpy="0 0 0" xyz="0.01 -0.045 0"/>
+                <geometry>
+                    <!-- <box size="0.03 0.09 0.01"/> -->
+                    <box size="0.02 0.07 0.01"/>
+                </geometry>
+                <!-- <origin rpy="0 0 0" xyz="0.01 -0.045 0"/> -->
+                <origin rpy="0 0 0" xyz="0.02 -0.045 0"/>
             </collision>
             <!-- Made up inertias from wrist -->
@@ -208,4 +212,5 @@
             <axis xyz="0 0 1"/>
             <limit effort="9.0" lower="0.0" upper = "6.2" velocity="0.5"/>
+            <dynamics damping="0.1" friction="0.1"/>
         </joint>
         <xacro:simple_transmission joint="${namespace}/joint1" />
@@ -216,4 +221,5 @@
             <axis xyz="0 0 1"/>
             <limit effort="9.0" lower="0.0" upper = "3.5" velocity="0.5"/>
+            <dynamics damping="0.1" friction="0.1"/>
         </joint>
         <xacro:simple_transmission joint="${namespace}/joint2" />
@@ -224,4 +230,5 @@
             <axis xyz="0 0 1"/>
             <limit effort="9.0" lower="0.0" upper = "3.5" velocity="0.5"/>
+            <dynamics damping="0.1" friction="0.1"/>
         </joint>
         <xacro:simple_transmission joint="${namespace}/joint3" />
@@ -232,4 +239,5 @@
             <axis xyz="0 0 1"/>
             <limit effort="5.0" lower="0.0" upper = "6.0" velocity="1.0"/>
+            <dynamics damping="0.1" friction="0.1"/>
         </joint>
         <xacro:simple_transmission joint="${namespace}/joint4" />
@@ -240,4 +248,5 @@
             <axis xyz="0 0 1"/>
             <limit effort="5.0" lower="0.0" upper = "0.5" velocity="0.5"/>
+            <dynamics damping="0.1" friction="0.1"/>
         </joint>
         <xacro:simple_transmission joint="${namespace}/joint5" />
@@ -248,4 +257,5 @@
             <axis xyz="0 0 -1"/>
             <limit effort="5.0" lower="0.0" upper = "0.5" velocity="0.5"/>
+            <dynamics damping="0.1" friction="0.1"/>
         </joint>
         <xacro:simple_transmission joint="${namespace}/joint6" />

File: seabotix_alpha_description/urdf/rexrov_oberon7.xacro (robot description, xacro)
@@ -19,5 +19,5 @@
   <xacro:include filename="$(find seabotix_alpha_description)/urdf/rexrov_base.xacro"/>
   <xacro:include filename="$(find seabotix_alpha_description)/urdf/rexrov.gazebo.xacro"/>
-  <xacro:include filename="$(find seabotix_alpha_description)/urdf/oberon7_default.xacro" />
+  <!-- <xacro:include filename="$(find seabotix_alpha_description)/urdf/oberon7_default.xacro" /> -->
   <xacro:include filename="$(find seabotix_alpha_description)/urdf/alpha_default.xacro" />
   <xacro:uuv_forward_looking_sonar
@@ -70,14 +70,14 @@
         <!-- Adding the hydrodynamic and hydrostatic parameters for the vehicle-->
         <xacro:rexrov_hydro_model namespace="$(arg namespace)"/>
-        <xacro:oberon7_hydro_model namespace="oberon7"/>
+        <!-- <xacro:oberon7_hydro_model namespace="oberon7"/> -->
         <xacro:alpha_hydro_model namespace="alpha"/>
       </plugin>
     </gazebo>
   </xacro:rexrov_base>
-  <xacro:oberon7 namespace="oberon7" parent="$(arg namespace)/base_link">
+  <!-- <xacro:oberon7 namespace="oberon7" parent="$(arg namespace)/base_link">
     <origin xyz="1.3 -0.5 -0.615" rpy="0 0 0"/>
-  </xacro:oberon7>
+  </xacro:oberon7> -->
   <xacro:alpha namespace="alpha" parent="$(arg namespace)/base_link">
-    <origin xyz="1.3 0.5 -0.615" rpy="0 0 0"/>
+    <origin xyz="0.3 0 0.1" rpy="0 0 0"/>
   </xacro:alpha>
   <gazebo>
