Commit message: Rename rexrov to seabotix
- Vehicle name changed to rexrov
- Moved worlds/rviz definition files into our package

File: seabotix_alpha_description/urdf/seabotix_alpha.xacro (robot description, xacro)
@@ -12,7 +12,7 @@
      limitations under the License.
 -->
-<robot name="rexrov" xmlns:xacro="http://www.ros.org/wiki/xacro" >
+<robot name="seabotix" xmlns:xacro="http://www.ros.org/wiki/xacro" >
   <xacro:arg name="debug" default="0"/>
-  <xacro:arg name="namespace" default="rexrov"/>
+  <xacro:arg name="namespace" default="seabotix"/>
   <xacro:arg name="inertial_reference_frame" default="world"/>
   <!-- Include the ROV macro file -->

File: seabotix_alpha_description/urdf/seabotix_base.xacro (robot description, xacro)
@@ -14,5 +14,5 @@
 <robot xmlns:xacro="http://www.ros.org/wiki/xacro">
   <!--
-      The RexROV meshes and hydrodynamic parameters are based on the parameters and dimensions
+      The Seabotix meshes and hydrodynamic parameters are based on the parameters and dimensions
       from the SF 30k.
       References:
@@ -26,5 +26,5 @@
   <xacro:include filename="$(find uuv_gazebo_ros_plugins)/urdf/snippets.xacro"/>
   <!-- Parameters -->
-  <xacro:property name="namespace" value="rexrov"/>
+  <xacro:property name="namespace" value="seabotix"/>
   <!-- <xacro:property name="visual_mesh_file" value="file://$(find uuv_descriptions)/meshes/RexROV_no_props.dae"/> -->
   <xacro:property name="visual_mesh_file" value="file://$(find seabotix_alpha_description)/meshes/seabotix.dae"/>
