Commit message: Add config files, Updat vehicle mesh w/o props
Added configuration files for thrusters and controllers
Added documentation on where to put said files
Updated the vehicle mesh to have holes where propellers should go

File: seabotix_alpha_description/urdf/seabotix_base.xacro (robot description, xacro)
@@ -27,6 +27,6 @@
   <!-- Parameters -->
   <xacro:property name="namespace" value="seabotix"/>
-  <!-- <xacro:property name="visual_mesh_file" value="file://$(find uuv_descriptions)/meshes/RexROV_no_props.dae"/> -->
-  <xacro:property name="visual_mesh_file" value="file://$(find seabotix_alpha_description)/meshes/seabotix.dae"/>
+  <xacro:property name="visual_mesh_file" value="file://$(find seabotix_alpha_description)/meshes/seabotix_no_props.dae"/>
+  <!-- <xacro:property name="visual_mesh_file" value="file://$(find seabotix_alpha_description)/meshes/seabotix.dae"/> -->
   <xacro:property name="prop_mesh_file" value="file://$(find seabotix_alpha_description)/meshes/prop.dae"/>
   <!-- Mass, see p.28 in Berg2012 -->
