Commit message: Thruster size/position/number updates
- Reduced thruster size to be reasonable for our vehicle
  (still need to check if it matches real life)
- Move thrusters to where they are located on the seabotix vehicle
- Removed extra thrusters that don't exist on our vehicle
- Updated thruster allocation matrix for new thruster set/location

File: seabotix_alpha_description/urdf/seabotix_actuators.xacro (robot description, xacro)
@@ -13,5 +13,5 @@
 -->
 <robot xmlns:xacro="http://www.ros.org/wiki/xacro">
-  <xacro:property name="prop_mesh_file" value="file://$(find seabotix_alpha_description)/meshes/prop.dae"/>
+  <xacro:property name="prop_mesh_file" value="file://$(find seabotix_alpha_description)/meshes/prop_scaled.dae"/>
   <!-- Thruster joint and link snippet -->
   <xacro:macro name="thruster_macro"
@@ -26,27 +26,32 @@
     </xacro:thruster_module_first_order_basic_fcn_macro>
   </xacro:macro>
+  <!-- Upper Left Thruster  -->
   <xacro:thruster_macro namespace="${namespace}" thruster_id="0">
-    <origin xyz="-0.890895 0.334385 0.528822" rpy="${0*d2r} ${-74.53*d2r} ${-53.21*d2r}"/>
+    <origin xyz="0 0.12 ${0.3-0.125}" rpy="0 -${pi/2} 0"/>
   </xacro:thruster_macro>
+  <!-- Upper Right Thruster -->
   <xacro:thruster_macro namespace="${namespace}" thruster_id="1">
-    <origin xyz="-0.890895 -0.334385 0.528822" rpy="${0*d2r} ${-74.53*d2r} ${53.21*d2r}"/>
+    <origin xyz="0 -0.12 ${0.3-0.125}" rpy="0 -${pi/2} 0"/>
   </xacro:thruster_macro>
+  <!-- SF fan -->
   <xacro:thruster_macro namespace="${namespace}" thruster_id="2">
-    <origin xyz="0.890895 0.334385 0.528822" rpy="${0*d2r} ${-105.47*d2r} ${53.21*d2r}"/>
+    <origin xyz="0.22 0.12 0" rpy="0 0 -${pi/4}"/>
   </xacro:thruster_macro>
+  <!-- PF fan -->
   <xacro:thruster_macro namespace="${namespace}" thruster_id="3">
-    <origin xyz="0.890895 -0.334385 0.528822" rpy="${0*d2r} ${-105.47*d2r} ${-53.21*d2r}"/>
+    <origin xyz="0.22 -0.12 0" rpy="0 0 ${pi/4}"/>  </xacro:thruster_macro>
+  <!-- SA fan -->
+  <xacro:thruster_macro namespace="${namespace}" thruster_id="4">
+    <origin xyz="-0.22 0.12 0" rpy="0 0 ${5*pi/4}"/>
   </xacro:thruster_macro>
-  <xacro:thruster_macro namespace="${namespace}" thruster_id="4">
-    <origin xyz="-0.412125 0.505415 0.129" rpy="${0*d2r} ${0*d2r} ${45*d2r}"/>
+  <!-- PA fan -->
+  <xacro:thruster_macro namespace="${namespace}" thruster_id="5">
+    <origin xyz="-0.22 -0.12 0" rpy="0 0 ${-5*pi/4}"/>
   </xacro:thruster_macro>
-  <xacro:thruster_macro namespace="${namespace}" thruster_id="5">
-    <origin xyz="-0.412125 -0.505415 0.129" rpy="${0*d2r} ${0*d2r} ${-45*d2r}"/>
-  </xacro:thruster_macro>
-  <xacro:thruster_macro namespace="${namespace}" thruster_id="6">
+  <!-- <xacro:thruster_macro namespace="${namespace}" thruster_id="6">
     <origin xyz="0.412125 0.505415 0.129" rpy="${0*d2r} ${0*d2r} ${135*d2r}"/>
   </xacro:thruster_macro>
   <xacro:thruster_macro namespace="${namespace}" thruster_id="7">
     <origin xyz="0.412125 -0.505415 0.129" rpy="${0*d2r} ${0*d2r} ${-135*d2r}"/>
-  </xacro:thruster_macro>
+  </xacro:thruster_macro> -->
 </robot>

File: seabotix_alpha_description/urdf/seabotix_base.xacro (robot description, xacro)
@@ -29,5 +29,5 @@
   <xacro:property name="visual_mesh_file" value="file://$(find seabotix_alpha_description)/meshes/seabotix_no_props.dae"/>
   <!-- <xacro:property name="visual_mesh_file" value="file://$(find seabotix_alpha_description)/meshes/seabotix.dae"/> -->
-  <xacro:property name="prop_mesh_file" value="file://$(find seabotix_alpha_description)/meshes/prop.dae"/>
+  <xacro:property name="prop_mesh_file" value="file://$(find seabotix_alpha_description)/meshes/prop_scale2.dae"/>
   <!-- Mass, see p.28 in Berg2012 -->
   <xacro:property name="mass" value="1862.87"/>
@@ -48,5 +48,5 @@
       </inertial>
       <visual>
-        <origin xyz="0 0 0" rpy="0 0 0"/>
+        <origin xyz="0 0 -0.125" rpy="0 0 0"/>
         <geometry>
           <mesh filename="${visual_mesh_file}" scale="1 1 1"/>

Commit message: Updated Inertia values for vehicle thruster
- Changed the inertia values in the thruster config files to match our vehicle
- Reduced mass of sonar that may have been throwing off center of mass
- Moved thrusters to be equally spaced in x/y plane

File: seabotix_alpha_description/urdf/seabotix_actuators.xacro (robot description, xacro)
@@ -36,16 +36,16 @@
   <!-- SF fan -->
   <xacro:thruster_macro namespace="${namespace}" thruster_id="2">
-    <origin xyz="0.22 0.12 0" rpy="0 0 -${pi/4}"/>
+    <origin xyz="0.12 0.12 0" rpy="0 0 -${pi/4}"/>
   </xacro:thruster_macro>
   <!-- PF fan -->
   <xacro:thruster_macro namespace="${namespace}" thruster_id="3">
-    <origin xyz="0.22 -0.12 0" rpy="0 0 ${pi/4}"/>  </xacro:thruster_macro>
+    <origin xyz="0.12 -0.12 0" rpy="0 0 ${pi/4}"/>  </xacro:thruster_macro>
   <!-- SA fan -->
   <xacro:thruster_macro namespace="${namespace}" thruster_id="4">
-    <origin xyz="-0.22 0.12 0" rpy="0 0 ${5*pi/4}"/>
+    <origin xyz="-0.12 0.12 0" rpy="0 0 ${5*pi/4}"/>
   </xacro:thruster_macro>
   <!-- PA fan -->
   <xacro:thruster_macro namespace="${namespace}" thruster_id="5">
-    <origin xyz="-0.22 -0.12 0" rpy="0 0 ${-5*pi/4}"/>
+    <origin xyz="-0.12 -0.12 0" rpy="0 0 ${-5*pi/4}"/>
   </xacro:thruster_macro>
   <!-- <xacro:thruster_macro namespace="${namespace}" thruster_id="6">

File: seabotix_alpha_description/urdf/seabotix_alpha.xacro (robot description, xacro)
@@ -25,5 +25,5 @@
       parent_link="${namespace}/base_link"
       topic="forward_sonar"
-      mass="0.015"
+      mass="0.0001"
       update_rate="40"
       samples="100"
@@ -31,7 +31,7 @@
         width="768"
         height="492">
-      <inertia ixx="0.00001" ixy="0.0" ixz="0.0" iyy="0.00001" iyz="0.0" izz="0.00001" />
+      <inertia ixx="0.000000007" ixy="0.0" ixz="0.0" iyy="0.000000007" iyz="0.0" izz="0.000000007" />
       <!--origin xyz="0.83 0 -0.22" rpy="0 ${0.2*pi} 0" /-->
-      <origin xyz="1.15 0 0.4" rpy="0 0.3 0"/>
+      <origin xyz="0 0 0" rpy="0 0.0 0"/>
       <visual>
       </visual>

File: seabotix_alpha_description/urdf/seabotix_base.xacro (robot description, xacro)
@@ -32,5 +32,5 @@
   <!-- <xacro:property name="mass" value="1862.87"/> -->
   <!-- <xacro:property name="mass" value="180.1"/> -->
-  <xacro:property name="mass" value="18.1"/>
+  <xacro:property name="mass" value="40.0"/>
   <xacro:property name="length" value="0.625"/>
   <xacro:property name="width" value="0.390"/>

Commit message: Updated Vehicle Thruster Placement/Collision
- Moved vehicle thrusters based on measurements from actual vehicle
- Adjusted collision envelope to match vehicle

File: seabotix_alpha_description/urdf/seabotix_actuators.xacro (robot description, xacro)
@@ -28,24 +28,24 @@
   <!-- Upper Left Thruster  -->
   <xacro:thruster_macro namespace="${namespace}" thruster_id="0">
-    <origin xyz="0 0.12 ${0.3-0.125}" rpy="0 -${pi/2} 0"/>
+    <origin xyz="0 0.12 ${0.3-0.125}" rpy="${-pi/3} ${-pi/3} ${-pi/2}"/>
   </xacro:thruster_macro>
   <!-- Upper Right Thruster -->
   <xacro:thruster_macro namespace="${namespace}" thruster_id="1">
-    <origin xyz="0 -0.12 ${0.3-0.125}" rpy="0 -${pi/2} 0"/>
+    <origin xyz="0 -0.12 ${0.3-0.125}" rpy="${pi/3} ${-pi/3} ${pi/2}"/>
   </xacro:thruster_macro>
   <!-- SF fan -->
   <xacro:thruster_macro namespace="${namespace}" thruster_id="2">
-    <origin xyz="0.12 0.12 0" rpy="0 0 -${pi/4}"/>
+    <origin xyz="0.2794 0.075 0" rpy="0 0 -${pi/4}"/>
   </xacro:thruster_macro>
   <!-- PF fan -->
   <xacro:thruster_macro namespace="${namespace}" thruster_id="3">
-    <origin xyz="0.12 -0.12 0" rpy="0 0 ${pi/4}"/>  </xacro:thruster_macro>
+    <origin xyz="0.2794 -0.075 0" rpy="0 0 ${pi/4}"/>  </xacro:thruster_macro>
   <!-- SA fan -->
   <xacro:thruster_macro namespace="${namespace}" thruster_id="4">
-    <origin xyz="-0.12 0.12 0" rpy="0 0 ${5*pi/4}"/>
+    <origin xyz="-0.2794 0.075 0" rpy="0 0 ${5*pi/4}"/>
   </xacro:thruster_macro>
   <!-- PA fan -->
   <xacro:thruster_macro namespace="${namespace}" thruster_id="5">
-    <origin xyz="-0.12 -0.12 0" rpy="0 0 ${-5*pi/4}"/>
+    <origin xyz="-0.2794 -0.075 0" rpy="0 0 ${-5*pi/4}"/>
   </xacro:thruster_macro>
   <!-- <xacro:thruster_macro namespace="${namespace}" thruster_id="6">

File: seabotix_alpha_description/urdf/seabotix_base.xacro (robot description, xacro)
@@ -34,7 +34,8 @@
   <xacro:property name="mass" value="40.0"/>
   <xacro:property name="mass_ratio" value="${40.0/1862.87}"/>
+<!-- Vehicle ~ 0.6096 m (2ft) x 0.4445 (17.5in) x 0.4572 (18in)-->
   <xacro:property name="length" value="0.625"/>
-  <xacro:property name="width" value="0.390"/>
-  <xacro:property name="height" value="0.390"/>
+  <xacro:property name="width" value="0.4572"/>
+  <xacro:property name="height" value="0.4572"/>
   <xacro:macro name="seabotix_base" params="namespace *gazebo inertial_reference_frame">
     <!-- base_link according to ROS conventions: x forward, z up -->
@@ -54,25 +55,31 @@
         </geometry>
       </visual>
-      <!-- bottom plate -->
       <collision>
-        <origin xyz="0 0 -0.75" rpy="0 0 0"/>
+        <origin xyz="0 0 0" rpy="0 0 0"/>
         <geometry>
-          <box size="2.56 1.50 0.10"/>
+          <box size="${length} ${width} ${height}"/>
         </geometry>
       </collision>
+      <!-- bottom plate -->
+      <!-- <collision>
+        <origin xyz="0 0 ${-height/2.0}" rpy="0 0 0"/>
+        <geometry>
+          <box size="${length} ${width+0.10} 0.10"/>
+        </geometry>
+      </collision> -->
       <!-- top plate -->
-      <collision>
-        <origin xyz="0 0 0.60" rpy="0 0 0"/>
-        <geometry><box size="2.56 1.50 0.40"/></geometry>
-      </collision>
+      <!-- <collision>
+        <origin xyz="0 0 ${height/2.0}" rpy="0 0 0"/>
+        <geometry><box size="${length} ${width+0.10} 0.10"/></geometry>
+      </collision> -->
       <!-- left / right sides -->
-      <collision>
-        <origin xyz="-0.20 0.70 -0.15" rpy="0 0 0"/>
-        <geometry><box size="2.20 0.10 1.10"/></geometry>
+      <!-- <collision>
+        <origin xyz="0 ${-width/2.0} 0" rpy="0 0 0"/>
+        <geometry><box size="${length} 0.10 ${height}"/></geometry>
       </collision>
       <collision>
-        <origin xyz="-0.20 -0.70 -0.15" rpy="0 0 0"/>
-        <geometry><box size="2.20 0.10 1.10"/></geometry>
-      </collision>
+        <origin xyz="0 ${width/2.0} 0" rpy="0 0 0"/>
+        <geometry><box size="${length} 0.10 ${height}"/></geometry>
+      </collision> -->
     </link>
     <!-- Set up hydrodynamic plugin given as input parameter -->
