Commit message: Renaming files to fit seabotix_alpha naming

File: seabotix_alpha_description/urdf/seabotix.gazebo.xacro (robot description, xacro)
@@ -21,5 +21,5 @@
     <!-- Volume, see p.31 in Berg2012 -->
     <xacro:property name="volume" value="1.83826"/>
-    <xacro:macro name="rexrov_hydro_model" params="namespace">
+    <xacro:macro name="seabotix_hydro_model" params="namespace">
         <link name="${namespace}/base_link">
             <neutrally_buoyant>0</neutrally_buoyant>

File: seabotix_alpha_description/urdf/seabotix_alpha.xacro (robot description, xacro)
@@ -17,7 +17,6 @@
   <xacro:arg name="inertial_reference_frame" default="world"/>
   <!-- Include the ROV macro file -->
-  <xacro:include filename="$(find seabotix_alpha_description)/urdf/rexrov_base.xacro"/>
-  <xacro:include filename="$(find seabotix_alpha_description)/urdf/rexrov.gazebo.xacro"/>
-  <!-- <xacro:include filename="$(find seabotix_alpha_description)/urdf/oberon7_default.xacro" /> -->
+  <xacro:include filename="$(find seabotix_alpha_description)/urdf/seabotix_base.xacro"/>
+  <xacro:include filename="$(find seabotix_alpha_description)/urdf/seabotix.gazebo.xacro"/>
   <xacro:include filename="$(find seabotix_alpha_description)/urdf/alpha_default.xacro" />
   <xacro:uuv_forward_looking_sonar
@@ -58,5 +57,5 @@
 -->
   <!-- Create the ROV -->
-  <xacro:rexrov_base
+  <xacro:seabotix_base
     namespace="$(arg namespace)"
     inertial_reference_frame="$(arg inertial_reference_frame)">
@@ -69,10 +68,10 @@
         <debug>$(arg debug)</debug>
         <!-- Adding the hydrodynamic and hydrostatic parameters for the vehicle-->
-        <xacro:rexrov_hydro_model namespace="$(arg namespace)"/>
+        <xacro:seabotix_hydro_model namespace="$(arg namespace)"/>
         <!-- <xacro:oberon7_hydro_model namespace="oberon7"/> -->
         <xacro:alpha_hydro_model namespace="alpha"/>
       </plugin>
     </gazebo>
-  </xacro:rexrov_base>
+  </xacro:seabotix_base>
   <!-- <xacro:oberon7 namespace="oberon7" parent="$(arg namespace)/base_link">
     <origin xyz="1.3 -0.5 -0.615" rpy="0 0 0"/>

File: seabotix_alpha_description/urdf/seabotix_base.xacro (robot description, xacro)
@@ -32,5 +32,9 @@
   <!-- Mass, see p.28 in Berg2012 -->
   <xacro:property name="mass" value="1862.87"/>
-  <xacro:macro name="rexrov_base" params="namespace *gazebo inertial_reference_frame">
+  <!-- <xacro:property name="mass" value="18.1"/> -->
+  <xacro:property name="length" value="0.625"/>
+  <xacro:property name="width" value="0.390"/>
+  <xacro:property name="height" value="0.390"/>
+  <xacro:macro name="seabotix_base" params="namespace *gazebo inertial_reference_frame">
     <!-- base_link according to ROS conventions: x forward, z up -->
     <link name="${namespace}/base_link">
@@ -39,4 +43,7 @@
         <origin xyz="0 0 0"/>
         <inertia ixx="525.39" ixy="1.44" ixz="33.41" iyy="794.20" iyz="2.6" izz="691.23"/>
+        <!-- <inertia ixx="${(1/3)*((length**2)+(height**2))*mass}" ixy="0.0" ixz="0.0"
+                 iyy="${(1/3)*((width**2)+(height**2))*mass}" iyz="0.0"
+                 izz="${(1/3)*((length**2)+(width**2))*mass}"/> -->
       </inertial>
       <visual>
@@ -76,6 +83,6 @@
       </plugin>
     </gazebo> -->
-    <xacro:include filename="$(find uuv_descriptions)/urdf/rexrov_actuators.xacro"/>
-    <xacro:include filename="$(find uuv_descriptions)/urdf/rexrov_sensors.xacro"/>
+    <xacro:include filename="$(find seabotix_alpha_description)/urdf/seabotix_actuators.xacro"/>
+    <xacro:include filename="$(find seabotix_alpha_description)/urdf/seabotix_sensors.xacro"/>
   </xacro:macro>
 </robot>

Commit message: Vehicle only launch files, tuning vehicle params
- Added launch files to only instantiate the vehicle.
- Updated mesh file for vehicle to include hole for second prop.
- Began tuning parameters for sensors.

File: seabotix_alpha_description/urdf/seabotix.gazebo.xacro (robot description, xacro)
@@ -18,15 +18,16 @@
     assume NWU (otherwise cob is below cog?).
     -->
-    <xacro:property name="cob" value="0.0 0.0 0.3"/>
+    <xacro:property name="cob" value="0.0 0.0 0.0"/>
     <!-- Volume, see p.31 in Berg2012 -->
-    <xacro:property name="volume" value="1.83826"/>
+    <!-- <xacro:property name="volume" value="1.83826"/> -->
+    <xacro:property name="volume" value="0.0951"/>
     <xacro:macro name="seabotix_hydro_model" params="namespace">
         <link name="${namespace}/base_link">
-            <neutrally_buoyant>0</neutrally_buoyant>
+            <neutrally_buoyant>1</neutrally_buoyant>
             <volume>${volume}</volume>
             <box>
-                <width>1.5</width>
-                <length>2.6</length>
-                <height>1.6</height>
+                <width>${width}</width>
+                <length>${length}</length>
+                <height>${height}</height>
             </box>
             <center_of_buoyancy>${cob}</center_of_buoyancy>
@@ -35,18 +36,18 @@
                 <!-- Added mass: see p.28 in Berg2012 -->
                 <added_mass>
-                     779.79 -6.8773 -103.32  8.5426 -165.54 -7.8033
-                    -6.8773    1222   51.29  409.44 -5.8488  62.726
-                    -103.32   51.29  3659.9  6.1112 -386.42  10.774
-                     8.5426  409.44  6.1112   534.9 -10.027  21.019
-                    -165.54 -5.8488 -386.42 -10.027  842.69 -1.1162
-                    -7.8033  62.726  10.775  21.019 -1.1162  224.32
+                    0 0 0 0 0 0
+                    0 0 0 0 0 0
+                    0 0 0 0 0 0
+                    0 0 0 0 0 0
+                    0 0 0 0 0 0
+                    0 0 0 0 0 0
                 </added_mass>
                 <!-- Linear damping: see p.31 in Berg2012 -->
                 <linear_damping>
-                    -74.82 -69.48 -728.4 -268.8 -309.77 -105
+                    0 0 0 0 0 0
                 </linear_damping>
                 <!-- Non-linear damping: see p.30 in Berg2012 -->
                 <quadratic_damping>
-                    -748.22 -992.53 -1821.01 -672 -774.44 -523.27
+                    0 0 0 0 0 0
                 </quadratic_damping>
             </hydrodynamic_model>

File: seabotix_alpha_description/urdf/seabotix_base.xacro (robot description, xacro)
@@ -29,8 +29,8 @@
   <xacro:property name="visual_mesh_file" value="file://$(find seabotix_alpha_description)/meshes/seabotix_no_props.dae"/>
   <!-- <xacro:property name="visual_mesh_file" value="file://$(find seabotix_alpha_description)/meshes/seabotix.dae"/> -->
-  <xacro:property name="prop_mesh_file" value="file://$(find seabotix_alpha_description)/meshes/prop_scale2.dae"/>
   <!-- Mass, see p.28 in Berg2012 -->
-  <xacro:property name="mass" value="1862.87"/>
-  <!-- <xacro:property name="mass" value="18.1"/> -->
+  <!-- <xacro:property name="mass" value="1862.87"/> -->
+  <!-- <xacro:property name="mass" value="180.1"/> -->
+  <xacro:property name="mass" value="18.1"/>
   <xacro:property name="length" value="0.625"/>
   <xacro:property name="width" value="0.390"/>
@@ -42,8 +42,8 @@
         <mass value="${mass}"/>
         <origin xyz="0 0 0"/>
-        <inertia ixx="525.39" ixy="1.44" ixz="33.41" iyy="794.20" iyz="2.6" izz="691.23"/>
-        <!-- <inertia ixx="${(1/3)*((length**2)+(height**2))*mass}" ixy="0.0" ixz="0.0"
+        <!-- <inertia ixx="525.39" ixy="1.44" ixz="33.41" iyy="794.20" iyz="2.6" izz="691.23"/> -->
+        <inertia ixx="${(1/3)*((length**2)+(height**2))*mass}" ixy="0.0" ixz="0.0"
                  iyy="${(1/3)*((width**2)+(height**2))*mass}" iyz="0.0"
-                 izz="${(1/3)*((length**2)+(width**2))*mass}"/> -->
+                 izz="${(1/3)*((length**2)+(width**2))*mass}"/>
       </inertial>
       <visual>

File: seabotix_alpha_description/urdf/seabotix_sensors.xacro (robot description, xacro)
@@ -18,5 +18,5 @@
     parent_link="${namespace}/base_link"
     inertial_reference_frame="${inertial_reference_frame}">
-    <origin xyz="-1.4 0 -0.312" rpy="0 ${0.5*pi} 0"/>
+    <origin xyz="0 0 0" rpy="0 0 0"/>
   </xacro:default_dvl_macro>
   <!-- Magnetometer  -->
@@ -24,9 +24,9 @@
   <!-- RPT  -->
   <xacro:default_rpt namespace="${namespace}" parent_link="${namespace}/base_link">
-    <origin xyz="-1.32 0 0.8" rpy="0 0 0"/>
+    <origin xyz="0 0 0" rpy="0 0 0"/>
   </xacro:default_rpt>
   <!-- Pressure  -->
   <xacro:default_pressure_macro namespace="${namespace}" parent_link="${namespace}/base_link">
-    <origin xyz="-1.32 0.5 0.85" rpy="0 0 0"/>
+    <origin xyz="0 0 0" rpy="0 0 0"/>
   </xacro:default_pressure_macro>
   <!-- IMU  -->
@@ -39,12 +39,12 @@
   <!-- Mount a camera -->
   <xacro:default_camera namespace="${namespace}" parent_link="${namespace}/base_link" suffix="">
-    <origin xyz="1.15 0 0.4" rpy="0 0.6 0"/>
+    <origin xyz="0 0 0" rpy="0 0 0"/>
   </xacro:default_camera>
-  <xacro:default_camera namespace="${namespace}" parent_link="${namespace}/base_link" suffix="right">
+  <!-- <xacro:default_camera namespace="${namespace}" parent_link="${namespace}/base_link" suffix="right">
     <origin xyz="1.15 -0.63 0.4" rpy="0 0.6 0.4"/>
-  </xacro:default_camera>
-  <xacro:default_camera namespace="${namespace}" parent_link="${namespace}/base_link" suffix="left">
+  </xacro:default_camera> -->
+  <!-- <xacro:default_camera namespace="${namespace}" parent_link="${namespace}/base_link" suffix="left">
     <origin xyz="1.15 0.63 0.4" rpy="0 0.6 -0.4"/>
-  </xacro:default_camera>
+  </xacro:default_camera> -->
   <!-- Mount a GPS. -->
   <xacro:default_gps namespace="${namespace}" parent_link="${namespace}/base_link" />

Commit message: Passive Stability, Damping Terms
- Made the vehicle passively stable by setting center of buoyancy
  above the center of gravity
- Added back the Added mass and damping terms from the RexRov vehicle,
  scaling them down by the ratio of the mass of the Seabotix vehicle
  to the mass of the Rexrov vehicle.
- These changes appear to alleviate the issue of the vehicle spinning
  out of control.

File: seabotix_alpha_description/urdf/seabotix.gazebo.xacro (robot description, xacro)
@@ -18,5 +18,5 @@
     assume NWU (otherwise cob is below cog?).
     -->
-    <xacro:property name="cob" value="0.0 0.0 0.0"/>
+    <xacro:property name="cob" value="0.0 0.0 0.05"/>
     <!-- Volume, see p.31 in Berg2012 -->
     <!-- <xacro:property name="volume" value="1.83826"/> -->
@@ -36,18 +36,18 @@
                 <!-- Added mass: see p.28 in Berg2012 -->
                 <added_mass>
-                    0 0 0 0 0 0
-                    0 0 0 0 0 0
-                    0 0 0 0 0 0
-                    0 0 0 0 0 0
-                    0 0 0 0 0 0
-                    0 0 0 0 0 0
+                    ${779.79*mass_ratio} ${-6.8773*mass_ratio} ${-103.32*mass_ratio}  ${8.5426*mass_ratio} ${-165.54*mass_ratio} ${-7.8033*mass_ratio}
+                    -${6.8773*mass_ratio}    ${1222*mass_ratio}   ${51.29*mass_ratio}  ${409.44*mass_ratio} ${-5.8488*mass_ratio}  ${62.726*mass_ratio}
+                    -${103.32*mass_ratio}   ${51.29*mass_ratio}  ${3659.9*mass_ratio}  ${6.1112*mass_ratio} ${-386.42*mass_ratio}  ${10.774*mass_ratio}
+                    ${8.5426*mass_ratio}  ${409.44*mass_ratio}  ${6.1112*mass_ratio}   ${534.9*mass_ratio} ${-10.027*mass_ratio}  ${21.019*mass_ratio}
+                    -${165.54*mass_ratio} ${-5.8488*mass_ratio} ${-386.42*mass_ratio} ${-10.027*mass_ratio}  ${842.69*mass_ratio} ${-1.1162*mass_ratio}
+                    -${7.8033*mass_ratio}  ${62.726*mass_ratio}  ${10.775*mass_ratio}  ${21.019*mass_ratio} ${-1.1162*mass_ratio}  ${224.32*mass_ratio}
                 </added_mass>
                 <!-- Linear damping: see p.31 in Berg2012 -->
                 <linear_damping>
-                    0 0 0 0 0 0
+                    ${-74.82*mass_ratio} ${-69.48*mass_ratio} ${-728.4*mass_ratio} ${-268.8*mass_ratio} ${-309.77*mass_ratio} ${-105*mass_ratio}
                 </linear_damping>
                 <!-- Non-linear damping: see p.30 in Berg2012 -->
                 <quadratic_damping>
-                    0 0 0 0 0 0
+                    ${-748.22*mass_ratio} ${-992.53*mass_ratio} ${-1821.01*mass_ratio} ${-672*mass_ratio} ${-774.44*mass_ratio} ${-523.27*mass_ratio}
                 </quadratic_damping>
             </hydrodynamic_model>

File: seabotix_alpha_description/urdf/seabotix_base.xacro (robot description, xacro)
@@ -30,7 +30,8 @@
   <!-- <xacro:property name="visual_mesh_file" value="file://$(find seabotix_alpha_description)/meshes/seabotix.dae"/> -->
   <!-- Mass, see p.28 in Berg2012 -->
-  <!-- <xacro:property name="mass" value="1862.87"/> -->
+  <xacro:property name="rexrov_mass" value="1862.87"/>
   <!-- <xacro:property name="mass" value="180.1"/> -->
   <xacro:property name="mass" value="40.0"/>
+  <xacro:property name="mass_ratio" value="${40.0/1862.87}"/>
   <xacro:property name="length" value="0.625"/>
   <xacro:property name="width" value="0.390"/>

Commit message: Moved Center of Buoyancy further up for more restoration forces

File: seabotix_alpha_description/urdf/seabotix.gazebo.xacro (robot description, xacro)
@@ -18,5 +18,5 @@
     assume NWU (otherwise cob is below cog?).
     -->
-    <xacro:property name="cob" value="0.0 0.0 0.05"/>
+    <xacro:property name="cob" value="0.0 0.0 0.1"/>
     <!-- Volume, see p.31 in Berg2012 -->
     <!-- <xacro:property name="volume" value="1.83826"/> -->

Commit message: Moved COB up more for potentially more stability
- COB = center of buoyancy

File: seabotix_alpha_description/urdf/seabotix.gazebo.xacro (robot description, xacro)
@@ -18,5 +18,5 @@
     assume NWU (otherwise cob is below cog?).
     -->
-    <xacro:property name="cob" value="0.0 0.0 0.1"/>
+    <xacro:property name="cob" value="0.0 0.0 0.5"/>
     <!-- Volume, see p.31 in Berg2012 -->
     <!-- <xacro:property name="volume" value="1.83826"/> -->

Commit message: Updated Turbulence Experiment
- Fixed logging information
- Ran some turbulence experiments and collected data

File: seabotix_alpha_description/urdf/seabotix.gazebo.xacro (robot description, xacro)
@@ -18,8 +18,8 @@
     assume NWU (otherwise cob is below cog?).
     -->
-    <xacro:property name="cob" value="0.0 0.0 0.5"/>
+    <xacro:property name="cob" value="0.0 0.0 0.05"/>
     <!-- Volume, see p.31 in Berg2012 -->
     <!-- <xacro:property name="volume" value="1.83826"/> -->
-    <xacro:property name="volume" value="0.0951"/>
+    <xacro:property name="volume" value="0.035"/>
     <xacro:macro name="seabotix_hydro_model" params="namespace">
         <link name="${namespace}/base_link">

Commit message: Updated Hydrodynamics Param (Stable at Spawn)
- Updated hydrodynamics parameters to better match seabotix vehicle
  based on Hannah's model
- Vehicle can be spawned stably using `roslaunch seabotix_alpha_description seabotix_vehicle.launch`
- However, moving the joystick around causes the vehicle to move uncontrollably
- Also vehicle still slightly sinks at start.

File: seabotix_alpha_description/urdf/seabotix.gazebo.xacro (robot description, xacro)
@@ -21,5 +21,5 @@
     <!-- Volume, see p.31 in Berg2012 -->
     <!-- <xacro:property name="volume" value="1.83826"/> -->
-    <xacro:property name="volume" value="0.035"/>
+    <xacro:property name="volume" value="0.0216"/>
     <xacro:macro name="seabotix_hydro_model" params="namespace">
         <link name="${namespace}/base_link">
@@ -36,18 +36,20 @@
                 <!-- Added mass: see p.28 in Berg2012 -->
                 <added_mass>
-                    ${779.79*mass_ratio} ${-6.8773*mass_ratio} ${-103.32*mass_ratio}  ${8.5426*mass_ratio} ${-165.54*mass_ratio} ${-7.8033*mass_ratio}
-                    -${6.8773*mass_ratio}    ${1222*mass_ratio}   ${51.29*mass_ratio}  ${409.44*mass_ratio} ${-5.8488*mass_ratio}  ${62.726*mass_ratio}
-                    -${103.32*mass_ratio}   ${51.29*mass_ratio}  ${3659.9*mass_ratio}  ${6.1112*mass_ratio} ${-386.42*mass_ratio}  ${10.774*mass_ratio}
-                    ${8.5426*mass_ratio}  ${409.44*mass_ratio}  ${6.1112*mass_ratio}   ${534.9*mass_ratio} ${-10.027*mass_ratio}  ${21.019*mass_ratio}
-                    -${165.54*mass_ratio} ${-5.8488*mass_ratio} ${-386.42*mass_ratio} ${-10.027*mass_ratio}  ${842.69*mass_ratio} ${-1.1162*mass_ratio}
-                    -${7.8033*mass_ratio}  ${62.726*mass_ratio}  ${10.775*mass_ratio}  ${21.019*mass_ratio} ${-1.1162*mass_ratio}  ${224.32*mass_ratio}
+                    8.10 -0.07 -1.07 0.09 -1.71 -0.08
+                    -0.07 12.69 0.53 4.25 -0.06 0.65
+                    -1.07 0.53 38.02 0.06 -4.01 0.11
+                    0.09 4.25 0.06 5.56 -0.10 0.22
+                    -1.71 -0.06 -4.01 -0.10 8.75 -0.01
+                    -0.08 0.65 0.11 0.22 -0.01 2.33
                 </added_mass>
-                <!-- Linear damping: see p.31 in Berg2012 -->
+                <!-- Linear damping: Hannah's values negated because these should be negative
+                for some reason -->
                 <linear_damping>
-                    ${-74.82*mass_ratio} ${-69.48*mass_ratio} ${-728.4*mass_ratio} ${-268.8*mass_ratio} ${-309.77*mass_ratio} ${-105*mass_ratio}
+                    -3.4 -4.6 -52.9 -4.5 -8.0 -2.7
                 </linear_damping>
-                <!-- Non-linear damping: see p.30 in Berg2012 -->
+                <!-- Linear damping: Hannah's values negated because these should be negative
+                for some reason -->
                 <quadratic_damping>
-                    ${-748.22*mass_ratio} ${-992.53*mass_ratio} ${-1821.01*mass_ratio} ${-672*mass_ratio} ${-774.44*mass_ratio} ${-523.27*mass_ratio}
+                    -34.4 -65.9 -132.3 -11.4 -20 -13.5
                 </quadratic_damping>
             </hydrodynamic_model>

File: seabotix_alpha_description/urdf/seabotix.xacro (robot description, xacro)
@@ -43,5 +43,5 @@
      allow the addition of external models of manipulator units -->
     <gazebo>
-      <plugin name="uuv_plugin" filename="libuuv_underwater_object_ros_plugin.so">
+      <plugin name="uuv_plugin_seabotix_base" filename="libuuv_underwater_object_ros_plugin.so">
         <fluid_density>1028.0</fluid_density>
         <flow_velocity_topic>hydrodynamics/current_velocity</flow_velocity_topic>

File: seabotix_alpha_description/urdf/seabotix_actuators.xacro (robot description, xacro)
@@ -28,24 +28,24 @@
   <!-- Upper Left Thruster  -->
   <xacro:thruster_macro namespace="${namespace}" thruster_id="0">
-    <origin xyz="0 0.12 ${0.3-0.125}" rpy="${-pi/3} ${-pi/3} ${-pi/2}"/>
+    <origin xyz="0 0.12 0.095" rpy="0 ${-pi/3} ${-pi/2}"/>
   </xacro:thruster_macro>
   <!-- Upper Right Thruster -->
   <xacro:thruster_macro namespace="${namespace}" thruster_id="1">
-    <origin xyz="0 -0.12 ${0.3-0.125}" rpy="${pi/3} ${-pi/3} ${pi/2}"/>
+    <origin xyz="0 -0.12 0.095" rpy="0 ${-pi/3} ${pi/2}"/>
   </xacro:thruster_macro>
   <!-- SF fan -->
   <xacro:thruster_macro namespace="${namespace}" thruster_id="2">
-    <origin xyz="0.2794 0.075 0" rpy="0 0 -${pi/4}"/>
+    <origin xyz="0.2794 0.075 -0.08" rpy="0 0 -${pi/4}"/>
   </xacro:thruster_macro>
   <!-- PF fan -->
   <xacro:thruster_macro namespace="${namespace}" thruster_id="3">
-    <origin xyz="0.2794 -0.075 0" rpy="0 0 ${pi/4}"/>  </xacro:thruster_macro>
+    <origin xyz="0.2794 -0.075 -0.08" rpy="0 0 ${pi/4}"/>  </xacro:thruster_macro>
   <!-- SA fan -->
   <xacro:thruster_macro namespace="${namespace}" thruster_id="4">
-    <origin xyz="-0.2794 0.075 0" rpy="0 0 ${5*pi/4}"/>
+    <origin xyz="-0.2794 0.075 -0.08" rpy="0 0 ${5*pi/4}"/>
   </xacro:thruster_macro>
   <!-- PA fan -->
   <xacro:thruster_macro namespace="${namespace}" thruster_id="5">
-    <origin xyz="-0.2794 -0.075 0" rpy="0 0 ${-5*pi/4}"/>
+    <origin xyz="-0.2794 -0.075 -0.08" rpy="0 0 ${-5*pi/4}"/>
   </xacro:thruster_macro>
   <!-- <xacro:thruster_macro namespace="${namespace}" thruster_id="6">

File: seabotix_alpha_description/urdf/seabotix_alpha.xacro (robot description, xacro)
@@ -63,5 +63,5 @@
      allow the addition of external models of manipulator units -->
     <gazebo>
-      <plugin name="uuv_plugin" filename="libuuv_underwater_object_ros_plugin.so">
+      <plugin name="uuv_plugin_seabotix_base" filename="libuuv_underwater_object_ros_plugin.so">
         <fluid_density>1028.0</fluid_density>
         <flow_velocity_topic>hydrodynamics/current_velocity</flow_velocity_topic>

File: seabotix_alpha_description/urdf/seabotix_base.xacro (robot description, xacro)
@@ -32,10 +32,10 @@
   <xacro:property name="rexrov_mass" value="1862.87"/>
   <!-- <xacro:property name="mass" value="180.1"/> -->
-  <xacro:property name="mass" value="40.0"/>
+  <xacro:property name="mass" value="22.2"/>
   <xacro:property name="mass_ratio" value="${40.0/1862.87}"/>
 <!-- Vehicle ~ 0.6096 m (2ft) x 0.4445 (17.5in) x 0.4572 (18in)-->
-  <xacro:property name="length" value="0.625"/>
-  <xacro:property name="width" value="0.4572"/>
-  <xacro:property name="height" value="0.4572"/>
+  <xacro:property name="length" value="0.64"/>
+  <xacro:property name="width" value="0.39"/>
+  <xacro:property name="height" value="0.39"/>
   <xacro:macro name="seabotix_base" params="namespace *gazebo inertial_reference_frame">
     <!-- Create a dummy link to avoid :KDL does not support a root link with an inertia warning. -->
@@ -47,7 +47,7 @@
         <origin xyz="0 0 0"/>
         <!-- <inertia ixx="525.39" ixy="1.44" ixz="33.41" iyy="794.20" iyz="2.6" izz="691.23"/> -->
-        <inertia ixx="${(1/3)*((length**2)+(height**2))*mass}" ixy="0.0" ixz="0.0"
-                 iyy="${(1/3)*((width**2)+(height**2))*mass}" iyz="0.0"
-                 izz="${(1/3)*((length**2)+(width**2))*mass}"/>
+        <inertia ixx="0.75" ixy="0.0" ixz="0.0"
+                 iyy="1.4" iyz="0.0"
+                 izz="1.6"/>
       </inertial>
       <visual>

Commit message: Modified volume for vehicle to not sink
- Set the neutrally buoyant flag for vehicle to 0 (because for some reason,
  vehicle still sinks even if the flag is set)
- Slightly increased volume of vehicle to be as expected
- Vehicle still suffering from unstable joystick control

File: seabotix_alpha_description/urdf/seabotix.gazebo.xacro (robot description, xacro)
@@ -21,8 +21,8 @@
     <!-- Volume, see p.31 in Berg2012 -->
     <!-- <xacro:property name="volume" value="1.83826"/> -->
-    <xacro:property name="volume" value="0.0216"/>
+    <xacro:property name="volume" value="0.02175"/>
     <xacro:macro name="seabotix_hydro_model" params="namespace">
         <link name="${namespace}/base_link">
-            <neutrally_buoyant>1</neutrally_buoyant>
+            <neutrally_buoyant>0</neutrally_buoyant>
             <volume>${volume}</volume>
             <box>
