Commit message: Moved arm URDF files to alpha_arm packaage
- Moved URDFs into the alpha_description package
- Changed references to arm URDFs to appropriate location

File: alpha_description/urdf/alpha_arm.gazebo.xacro (robot description, xacro)
@@ -1,5 +1,5 @@
 <?xml version="1.0"?>
 <robot xmlns:xacro="http://www.ros.org/wiki/xacro">
-  <xacro:include filename="$(find seabotix_alpha_description)/urdf/alpha_arm_ft_sensor.xacro" />
+  <xacro:include filename="$(find alpha_description)/urdf/alpha_arm_ft_sensor.xacro" />
   <xacro:macro name="alpha_gazebo_macro" params="namespace">
     <gazebo reference="${namespace}/base_link">

File: alpha_description/urdf/alpha_arm.xacro (robot description, xacro)
@@ -33,23 +33,23 @@
         <link name="${namespace}/base_link">
             <visual>
-            <geometry>
-            <mesh filename="package://reach_system_one_support/meshes/reach5mini/visual/Base.stl" />
-            </geometry>
-            <origin rpy="0 0 0" xyz="0 0 0"/>
-            <material name="black_arm"/>
-            </visual>
-            <collision>
-            <geometry>
-                <cylinder length="0.150" radius="0.020"/>
-            </geometry>
-            <origin rpy="0 1.57075 0" xyz="-0.075 0 0"/>
-            </collision>
-            <inertial>
-            <mass value="0.341"/>
-            <origin xyz="-0.075 -0.006 -0.003"/>
-            <inertia ixx="0.000099" ixy="0.000139" ixz="0.000115" iyy="0.002920" iyz="0.000003" izz="0.002934"/>
-            <!-- <inertia ixx="${(1/12)*0.341*(0.150)**2 + 0.25*0.341*0.020**2}" ixy="0.0" ixz="0.0"
-            iyy="${(1/12)*0.341*(0.150)**2 + 0.25*0.341*0.020**2}" iyz="0.0"
-            izz="${0.5*0.341*0.020**2}"/> -->
+                <geometry>
+                    <mesh filename="package://reach_system_one_support/meshes/reach5mini/visual/Base.stl" />
+                </geometry>
+                <origin rpy="0 0 0" xyz="0 0 0"/>
+                <material name="black_arm"/>
+            </visual>
+            <collision>
+                <geometry>
+                    <cylinder length="0.150" radius="0.020"/>
+                </geometry>
+                <origin rpy="0 1.57075 0" xyz="-0.075 0 0"/>
+            </collision>
+            <inertial>
+                <mass value="0.341"/>
+                <origin xyz="-0.075 -0.006 -0.003"/>
+                <inertia ixx="0.000099" ixy="0.000139" ixz="0.000115" iyy="0.002920" iyz="0.000003" izz="0.002934"/>
+                <!-- <inertia ixx="${(1/12)*0.341*(0.150)**2 + 0.25*0.341*0.020**2}" ixy="0.0" ixz="0.0"
+                iyy="${(1/12)*0.341*(0.150)**2 + 0.25*0.341*0.020**2}" iyz="0.0"
+                izz="${0.5*0.341*0.020**2}"/> -->
             </inertial>
         </link>

File: alpha_description/urdf/alpha_default.xacro (robot description, xacro)
@@ -14,7 +14,7 @@
 <robot name="alpha" xmlns:xacro="http://www.ros.org/wiki/xacro">
   <!-- Import serial arm -->
-  <xacro:include filename="$(find seabotix_alpha_description)/urdf/alpha_arm.xacro" />
+  <xacro:include filename="$(find alpha_description)/urdf/alpha_arm.xacro" />
   <!-- Import Gazebo specific macros -->
-  <xacro:include filename="$(find seabotix_alpha_description)/urdf/alpha_arm.gazebo.xacro" />
+  <xacro:include filename="$(find alpha_description)/urdf/alpha_arm.gazebo.xacro" />
   <xacro:macro name="alpha" params="namespace parent *origin">
     <xacro:alpha_arm namespace="${namespace}"/>

File: seabotix_alpha_description/urdf/seabotix_alpha.xacro (robot description, xacro)
@@ -19,5 +19,5 @@
   <xacro:include filename="$(find seabotix_alpha_description)/urdf/seabotix_base.xacro"/>
   <xacro:include filename="$(find seabotix_alpha_description)/urdf/seabotix.gazebo.xacro"/>
-  <xacro:include filename="$(find seabotix_alpha_description)/urdf/alpha_default.xacro" />
+  <xacro:include filename="$(find alpha_description)/urdf/alpha_default.xacro" />
   <xacro:uuv_forward_looking_sonar
       namespace="${namespace}"
@@ -78,5 +78,5 @@
   </xacro:oberon7> -->
   <xacro:alpha namespace="alpha" parent="$(arg namespace)/base_link">
-    <origin xyz="0.3 0 0.1" rpy="0 0 0"/>
+    <origin xyz="0.0 0 -${height/2}" rpy="0 ${pi/2} 0"/>
   </xacro:alpha>
   <gazebo>
