Commit message: Fixed Joint Limits
- Fixed Joint limits for certain joints that seemed unrealistic
  based on arm positioning. They may actually be correct, so check
  once the hardware gets here.

File: alpha_description/urdf/alpha_arm.xacro (robot description, xacro)
@@ -34,5 +34,5 @@
             <visual>
                 <geometry>
-                    <mesh filename="package://reach_system_one_support/meshes/reach5mini/visual/Base.stl" />
+                    <mesh filename="package://alpha_description/meshes/reach5mini/visual/Base.stl" />
                 </geometry>
                 <origin rpy="0 0 0" xyz="0 0 0"/>
@@ -57,5 +57,5 @@
             <visual>
             <geometry>
-                <mesh filename="package://reach_system_one_support/meshes/reach5mini/visual/ShoulderJoint.stl" />
+                <mesh filename="package://alpha_description/meshes/reach5mini/visual/ShoulderJoint.stl" />
             </geometry>
             <material name="black_arm"/>
@@ -80,5 +80,5 @@
             <visual>
             <geometry>
-                <mesh filename="package://reach_system_one_support/meshes/reach5mini/visual/UpperArm.stl" />
+                <mesh filename="package://alpha_description/meshes/reach5mini/visual/UpperArm.stl" />
             </geometry>
             <origin rpy="0 -1.57075 -0.2655555" xyz="0 0 -0.075"/>
@@ -109,5 +109,5 @@
             <visual>
             <geometry>
-                <mesh filename="package://reach_system_one_support/meshes/reach5mini/visual/ForearmJoint.stl" />
+                <mesh filename="package://alpha_description/meshes/reach5mini/visual/ForearmJoint.stl" />
             </geometry>
             <origin rpy="0 0 0" xyz="0 0 0"/>
@@ -132,5 +132,5 @@
             <visual>
             <geometry>
-                <mesh filename="package://reach_system_one_support/meshes/reach5mini/visual/Wrist.stl" />
+                <mesh filename="package://alpha_description/meshes/reach5mini/visual/Wrist.stl" />
             </geometry>
             <origin rpy="0 0 0" xyz="0 0 0"/>
@@ -157,5 +157,5 @@
             <visual>
                 <geometry>
-                    <mesh filename="package://reach_system_one_support/meshes/reach5mini/visual/Jaw1.stl" />
+                    <mesh filename="package://alpha_description/meshes/reach5mini/visual/Jaw1.stl" />
                 </geometry>
                 <origin rpy="0 0 0" xyz="0 0 0"/>
@@ -164,10 +164,17 @@
             <collision>
                 <geometry>
-                    <!-- <box size="0.03 0.09 0.01"/> -->
+                    <mesh filename="package://alpha_description/meshes/reach5mini/visual/Jaw1.stl" scale="1 1 0.9"/>
+                </geometry>
+            </collision>
+            <!-- <collision> -->
+                <!-- <origin rpy="0 0 0" xyz="0 0 0"/> -->
+                <!-- <geometry>
+                    <mesh filename="package://alpha_description/meshes/reach5mini/visual/Jaw1.stl" scale="1 1 0.9"/>
+                </geometry>                 -->
+                <!-- <geometry>
                     <box size="0.02 0.07 0.01"/>
                 </geometry>
-                <!-- <origin rpy="0 0 0" xyz="-0.01 -0.045 0"/> -->
-                <origin rpy="0 0 0" xyz="-0.02 -0.045 0"/>
-            </collision>
+                <origin rpy="0 0 0" xyz="-0.04 -0.045 0"/> -->
+            <!-- </collision> -->
             <!-- Made up inertias from wrist -->
             <inertial>
@@ -182,18 +189,26 @@
         <link name="${namespace}/jaw2">
             <visual>
-            <geometry>
-                <mesh filename="package://reach_system_one_support/meshes/reach5mini/visual/Jaw2.stl" />
-            </geometry>
-            <origin rpy="0 0 0" xyz="0 0 0"/>
-            <material name="black_arm"/>
-            </visual>
-            <collision>
-                <geometry>
-                    <!-- <box size="0.03 0.09 0.01"/> -->
+                <geometry>
+                    <mesh filename="package://alpha_description/meshes/reach5mini/visual/Jaw2.stl" />
+                </geometry>
+                <origin rpy="0 0 0" xyz="0 0 0"/>
+                <material name="black_arm"/>
+            </visual>
+            <collision>
+                <geometry>
+                    <mesh filename="package://alpha_description/meshes/reach5mini/visual/Jaw2.stl" scale="1 1 0.9"/>
+                </geometry>
+            </collision>
+            <!-- <collision> -->
+                <!-- <geometry>
+                    <mesh filename="package://alpha_description/meshes/reach5mini/visual/Jaw2.stl" scale="1 1 0.9"/>
+                </geometry> -->
+                <!-- <origin rpy="0 0 0" xyz="0 0 0"/>
+                <geometry>
                     <box size="0.02 0.07 0.01"/>
                 </geometry>
-                <!-- <origin rpy="0 0 0" xyz="0.01 -0.045 0"/> -->
-                <origin rpy="0 0 0" xyz="0.02 -0.045 0"/>
-            </collision>
+                <origin rpy="0 0 0" xyz="0.01 -0.045 0"/>
+                <origin rpy="0 0 0" xyz="0.04 -0.045 0"/> -->
+            <!-- </collision> -->
             <!-- Made up inertias from wrist -->
             <inertial>
@@ -211,5 +226,5 @@
             <origin xyz="0 0 0" rpy="0 0 0"/> <!--Was <origin xyz="0 0 0" rpy="0 0 3.141592/> before-->
             <axis xyz="0 0 1"/>
-            <limit effort="9.0" lower="0.0" upper = "6.2" velocity="0.5"/>
+            <limit effort="9.0" lower="-${pi}" upper = "${pi}" velocity="0.5"/>
             <dynamics damping="0.1" friction="0.1"/>
         </joint>
@@ -238,5 +253,5 @@
             <origin xyz="0.020 0 0" rpy="-1.57075 0 0"/>
             <axis xyz="0 0 1"/>
-            <limit effort="5.0" lower="0.0" upper = "6.0" velocity="1.0"/>
+            <limit effort="5.0" lower="${-pi}" upper = "${pi}" velocity="1.0"/>
             <dynamics damping="0.1" friction="0.1"/>
         </joint>

Commit message: Alpha Arm Outreached poses / Updated Rviz launch
- Added commented out sections to the Alpha Arm URDF that denote
  the transforms to have the arm begin in an outstretched position
- Updated Rviz launch parameters

File: alpha_description/urdf/alpha_arm.xacro (robot description, xacro)
@@ -219,5 +219,5 @@
             iyy="${1/12*0.333*(0.03**2+0.01**2)}" iyz="0.0"
             izz="${1/12*0.333*(0.03**2+0.09**2)}"/>
-            </inertial>-->
+            </inertial>
         </link>
         <joint name="${namespace}/joint1" type="revolute">
@@ -232,6 +232,6 @@
         <joint name="${namespace}/joint2" type="revolute">
             <parent link="${namespace}/shoulder_link"/>
-            <child link="${namespace}/upper_arm_link"/>
-            <origin xyz="0.020 0 0.046" rpy="1.57075 1.3 0"/>
+            <child link="${namespace}/upper_arm_link"/>            <origin xyz="0.020 0 0.046" rpy="1.57075 1.3 0"/>
+            <!-- <origin xyz="0.020 0 0.046" rpy="1.57075 0 0"/> -->
             <axis xyz="0 0 1"/>
             <limit effort="9.0" lower="0.0" upper = "3.5" velocity="0.5"/>
@@ -243,4 +243,5 @@
             <child link="${namespace}/forearm_link"/>
             <origin xyz="0.15 0 0" rpy="3.1415 0 1.3"/>
+            <!-- <origin xyz="0.15 0 0" rpy="3.1415 0 ${-pi/2}"/> -->
             <axis xyz="0 0 1"/>
             <limit effort="9.0" lower="0.0" upper = "3.5" velocity="0.5"/>

Commit message: Reran Moveit Setup, Updated Kinematic xacro
- Updated the xacro file for the kinematic version of uvms
  which contains both the arm and vehicle in the same urdf for planning
- Reran Moveit setup with vehicle

TODO:
- We seemed to have a regression where we can only generate plans for
  the arm and not the vehicle.
- Need to check for the cause of this regression.
- Placement of arm in vehicle URDF may be slightly different from
  actual vehicle due to differing origins
- Need to match namespacing between kinematic xacro and Project Dave video

File: alpha_description/urdf/alpha_arm.xacro (robot description, xacro)
@@ -232,5 +232,6 @@
         <joint name="${namespace}/joint2" type="revolute">
             <parent link="${namespace}/shoulder_link"/>
-            <child link="${namespace}/upper_arm_link"/>            <origin xyz="0.020 0 0.046" rpy="1.57075 1.3 0"/>
+            <child link="${namespace}/upper_arm_link"/>
+            <origin xyz="0.020 0 0.046" rpy="1.57075 1.3 0"/>
             <!-- <origin xyz="0.020 0 0.046" rpy="1.57075 0 0"/> -->
             <axis xyz="0 0 1"/>
@@ -262,4 +263,5 @@
             <child link="${namespace}/jaw1"/>
             <origin xyz="0.015 0 -0.140" rpy="1.57075 0 0"/>
+            <!-- was <axis xyz="0 0 -1"/> in original urdf -->
             <axis xyz="0 0 1"/>
             <limit effort="5.0" lower="0.0" upper = "0.5" velocity="0.5"/>

File: seabotix_alpha_description/urdf/seabotix_alpha.xacro (robot description, xacro)
@@ -77,4 +77,5 @@
     <origin xyz="1.3 -0.5 -0.615" rpy="0 0 0"/>
   </xacro:oberon7> -->
+  <!-- height xacro parameter defined in seabotix_base.xacro -->
   <xacro:alpha namespace="alpha" parent="$(arg namespace)/base_link">
     <origin xyz="0.0 0 -${height/2}" rpy="0 ${pi/2} 0"/>

File: seabotix_alpha_description/urdf/seabotix_alpha_kinematic.xacro (robot description, xacro)
@@ -11,4 +11,8 @@
   <!-- Fluid density -->
   <xacro:property name="rho" value="1028"/>
+<!-- Vehicle ~ 0.6096 m (2ft) x 0.4445 (17.5in) x 0.4572 (18in)-->
+  <xacro:property name="length" value="0.625"/>
+  <xacro:property name="width" value="0.4572"/>
+  <xacro:property name="height" value="0.4572"/>
   <!--
     Visual mesh file for the vehicle, usually in DAE (Collada) format. Be sure to store the
@@ -587,5 +591,5 @@
     <origin xyz="0 0 0" rpy="0 0 0"/> <!--Was <origin xyz="0 0 0" rpy="0 0 3.141592/> before-->
     <axis xyz="0 0 1"/>
-    <limit effort="9.0" lower="0.0" upper = "6.2" velocity="0.5"/>
+    <limit effort="9.0" lower="-${pi}" upper = "${pi}" velocity="0.5"/>
   </joint>
   <joint name="joint2" type="revolute">
@@ -608,5 +612,5 @@
     <origin xyz="0.020 0 0" rpy="-1.57075 0 0"/>
     <axis xyz="0 0 1"/>
-    <limit effort="5.0" lower="0.0" upper = "6.0" velocity="1.0"/>
+            <limit effort="5.0" lower="${-pi}" upper = "${pi}" velocity="1.0"/>
   </joint>
   <joint name="joint5" type="revolute">
@@ -683,5 +687,5 @@
       <parent link="world_link_yaw"/>
       <child link="arm_base_link"/>
-      <origin rpy="0 0 0" xyz="${0.25 + 0.075 + 0.075 +0.05} 0 0"/>
+      <origin xyz="0.0 0 -${3*height/4}" rpy="0 ${pi/2} 0"/>
     </joint>
     <!-- <gazebo reference="${namespace}/base_link"> -->

Commit message: Moved Controller Config, Kinematic URDF Namespace
- Moved controller config for the arm to its own folder
- Edited the kinematic URDF of the UVMS system to reflect
  the state of the xacro file

File: alpha_description/urdf/alpha_arm.xacro (robot description, xacro)
@@ -263,5 +263,4 @@
             <child link="${namespace}/jaw1"/>
             <origin xyz="0.015 0 -0.140" rpy="1.57075 0 0"/>
-            <!-- was <axis xyz="0 0 -1"/> in original urdf -->
             <axis xyz="0 0 1"/>
             <limit effort="5.0" lower="0.0" upper = "0.5" velocity="0.5"/>

File: seabotix_alpha_description/urdf/seabotix_alpha_kinematic.xacro (robot description, xacro)
@@ -15,4 +15,7 @@
   <xacro:property name="width" value="0.4572"/>
   <xacro:property name="height" value="0.4572"/>
+  <!-- The namespace_arm for the seabotix alpha arm -->
+  <xacro:property name="namespace_vehicle" value="seabotix"/>
+  <xacro:property name="namespace_arm" value="${namespace_vehicle}/alpha"/>
   <!--
     Visual mesh file for the vehicle, usually in DAE (Collada) format. Be sure to store the
@@ -30,5 +33,5 @@
   -->
   <!-- Vehicle macro -->
-  <!-- <xacro:macro name="seabotix_alpha_base" params="namespace *gazebo"> -->
+  <!-- <xacro:macro name="seabotix_alpha_base" params="namespace_arm *gazebo"> -->
     <link name="base_link">
         <inertial>
@@ -42,5 +45,5 @@
     <link name="world_link_x">
         <inertial>
-        <mass value="${mass}" />
+        <mass value="0" />
         <origin xyz="${cog}" rpy="0 0 0"/>
         <inertia ixx="0" ixy="0" ixz="0"
@@ -51,5 +54,5 @@
     <link name="world_link_y">
         <inertial>
-        <mass value="${mass}" />
+        <mass value="0" />
         <origin xyz="${cog}" rpy="0 0 0"/>
         <inertia ixx="0" ixy="0" ixz="0"
@@ -60,5 +63,5 @@
     <link name="world_link_z">
         <inertial>
-        <mass value="${mass}" />
+        <mass value="0" />
         <origin xyz="${cog}" rpy="0 0 0"/>
         <inertia ixx="0" ixy="0" ixz="0"
@@ -69,5 +72,5 @@
     <link name="world_link_roll">
         <inertial>
-        <mass value="${mass}" />
+        <mass value="0" />
         <origin xyz="${cog}" rpy="0 0 0"/>
         <inertia ixx="0" ixy="0" ixz="0"
@@ -78,5 +81,5 @@
     <link name="world_link_pitch">
         <inertial>
-        <mass value="${mass}" />
+        <mass value="0" />
         <origin xyz="${cog}" rpy="0 0 0"/>
         <inertia ixx="0" ixy="0" ixz="0"
@@ -86,5 +89,5 @@
     </link>
       <!-- Rigid body description of the base link -->
-      <!-- <link name="${namespace}/base_link"> -->
+      <!-- <link name="${namespace_arm}/base_link"> -->
       <link name="world_link_yaw">
         <!--
@@ -115,5 +118,5 @@
       </link>
       <!-- robot name="OSU vLBV300 Volturnus" -->
-      <xacro:property name="pi" value="3.1515926535897931" />
+      <!-- <xacro:property name="pi" value="3.1515926535897931" /> -->
       <xacro:property name="deg2rad" value="${pi/180}" />
       <!-- Without trig, angles are a pain in the arse. Beam angle 30 -->
@@ -448,5 +451,5 @@
       </joint>
 <!-- Reach 5 Arm -->
-  <link name="arm_base_link">
+  <link name="${namespace_arm}/base_link">
     <visual>
       <geometry>
@@ -468,5 +471,5 @@
     </inertial>
   </link>
-  <link name="shoulder_link">
+  <link name="${namespace_arm}/shoulder_link">
     <visual>
       <geometry>
@@ -488,5 +491,5 @@
     </inertial>
   </link>
-  <link name="upper_arm_link">
+  <link name="${namespace_arm}/upper_arm_link">
     <visual>
       <geometry>
@@ -514,5 +517,5 @@
     </inertial>
   </link>
-  <link name="forearm_link">
+  <link name="${namespace_arm}/forearm_link">
     <visual>
       <geometry>
@@ -534,5 +537,5 @@
     </inertial>
   </link>
-  <link name="wrist_link">
+  <link name="${namespace_arm}/wrist_link">
     <visual>
       <geometry>
@@ -554,7 +557,7 @@
     </inertial>
   </link>
-  <link name="tip">
+  <link name="${namespace_arm}/tip">
   </link>
-  <link name="jaw1">
+  <link name="${namespace_arm}/jaw1">
     <visual>
       <geometry>
@@ -571,5 +574,5 @@
     </collision>
   </link>
-  <link name="jaw2">
+  <link name="${namespace_arm}/jaw2">
     <visual>
       <geometry>
@@ -586,49 +589,49 @@
     </collision>
   </link>
-  <joint name="joint1" type="revolute">
-    <parent link="arm_base_link"/>
-    <child link="shoulder_link"/>
+  <joint name="${namespace_arm}/joint1" type="revolute">
+    <parent link="${namespace_arm}/base_link"/>
+    <child link="${namespace_arm}/shoulder_link"/>
     <origin xyz="0 0 0" rpy="0 0 0"/> <!--Was <origin xyz="0 0 0" rpy="0 0 3.141592/> before-->
     <axis xyz="0 0 1"/>
     <limit effort="9.0" lower="-${pi}" upper = "${pi}" velocity="0.5"/>
   </joint>
-  <joint name="joint2" type="revolute">
-    <parent link="shoulder_link"/>
-    <child link="upper_arm_link"/>
+  <joint name="${namespace_arm}/joint2" type="revolute">
+    <parent link="${namespace_arm}/shoulder_link"/>
+    <child link="${namespace_arm}/upper_arm_link"/>
     <origin xyz="0.020 0 0.046" rpy="1.57075 1.3 0"/>
     <axis xyz="0 0 1"/>
     <limit effort="9.0" lower="0.0" upper = "3.5" velocity="0.5"/>
   </joint>
-  <joint name="joint3" type="revolute">
-    <parent link="upper_arm_link"/>
-    <child link="forearm_link"/>
+  <joint name="${namespace_arm}/joint3" type="revolute">
+    <parent link="${namespace_arm}/upper_arm_link"/>
+    <child link="${namespace_arm}/forearm_link"/>
     <origin xyz="0.15 0 0" rpy="3.1415 0 1.3"/>
     <axis xyz="0 0 1"/>
     <limit effort="9.0" lower="0.0" upper = "3.5" velocity="0.5"/>
   </joint>
-  <joint name="joint4" type="revolute">
-    <parent link="forearm_link"/>
-    <child link="wrist_link"/>
+  <joint name="${namespace_arm}/joint4" type="revolute">
+    <parent link="${namespace_arm}/forearm_link"/>
+    <child link="${namespace_arm}/wrist_link"/>
     <origin xyz="0.020 0 0" rpy="-1.57075 0 0"/>
     <axis xyz="0 0 1"/>
             <limit effort="5.0" lower="${-pi}" upper = "${pi}" velocity="1.0"/>
   </joint>
-  <joint name="joint5" type="revolute">
-    <parent link="wrist_link"/>
-    <child link="jaw1"/>
+  <joint name="${namespace_arm}/joint5" type="revolute">
+    <parent link="${namespace_arm}/wrist_link"/>
+    <child link="${namespace_arm}/jaw1"/>
     <origin xyz="0.015 0 -0.140" rpy="1.57075 0 0"/>
     <axis xyz="0 0 1"/>
     <limit effort="5.0" lower="0.0" upper = "0.5" velocity="0.5"/>
   </joint>
-  <joint name="joint6" type="revolute">
-    <parent link="wrist_link"/>
-    <child link="jaw2"/>
+  <joint name="${namespace_arm}/joint6" type="revolute">
+    <parent link="${namespace_arm}/wrist_link"/>
+    <child link="${namespace_arm}/jaw2"/>
     <origin xyz="-0.015 0 -0.140" rpy="1.57075 0 0"/>
     <axis xyz="0 0 -1"/>
     <limit effort="5.0" lower="0.0" upper = "0.5" velocity="0.5"/>
   </joint>
-  <joint name="arm_to_tip" type="fixed">
-    <parent link="wrist_link"/>
-    <child link="tip"/>
+  <joint name="${namespace_arm}/arm_to_tip" type="fixed">
+    <parent link="${namespace_arm}/wrist_link"/>
+    <child link="${namespace_arm}/tip"/>
     <origin xyz="0 0 -0.180" rpy="0 1.57075 0"/>
   </joint>
@@ -654,17 +657,19 @@
       <limit effort="100" velocity="0.5" lower="-10" upper="10" /> <!-- Assume we are operating in 20x20x20m cube-->
     </joint>
-    <joint name="roll_displacement" type="revolute">
+    <joint name="roll_displacement" type="fixed">
       <parent link="world_link_z"/>
       <child link="world_link_roll"/>
       <origin rpy="0 0 0" xyz="0 0 0"/>
-      <axis xyz="1 0 0"/>
-      <limit effort="100" velocity="${pi/10}" lower="${-pi/2}" upper="${pi/2}" /> <!-- Assume we can roll by pi/2-->
+      <!-- <axis xyz="1 0 0"/> -->
+      <!-- <limit effort="100" velocity="${pi/10}" lower="${-pi/2}" upper="${pi/2}" />  -->
+      <!-- Assume we can roll by pi/2-->
     </joint>
-    <joint name="pitch_displacement" type="revolute">
+    <joint name="pitch_displacement" type="fixed">
       <parent link="world_link_roll"/>
       <child link="world_link_pitch"/>
       <origin rpy="0 0 0" xyz="0 0 0"/>
       <axis xyz="0 1 0"/>
-      <limit effort="100" velocity="${pi/10}" lower="${-pi/2}" upper="${pi/2}" /> <!-- Assume we can pitch by pi/2-->
+      <!-- <limit effort="100" velocity="${pi/10}" lower="${-pi/2}" upper="${pi/2}" />  -->
+      <!-- Assume we can pitch by pi/2-->
     </joint>
     <joint name="yaw_displacement" type="continuous">
@@ -677,5 +682,5 @@
     <!-- Add a link attaching the vehicle to the world base link -->
     <joint name="joint_vehicle_base_world" type="fixed">
-      <!-- <parent link="${namespace}/base_link"/> -->
+      <!-- <parent link="${namespace_arm}/base_link"/> -->
       <parent link="world_link_yaw"/>
       <child link="vehicle_base_link"/>
@@ -683,11 +688,11 @@
     </joint>
     <!-- Add a link attaching the arm to the world base link -->
-    <joint name="joint_arm_base_world" type="fixed">
-      <!-- <parent link="${namespace}/base_link"/> -->
-      <parent link="world_link_yaw"/>
-      <child link="arm_base_link"/>
+    <joint name="joint_arm_vehicle" type="fixed">
+      <!-- <parent link="${namespace_arm}/base_link"/> -->
+      <parent link="vehicle_base_link"/>
+      <child link="${namespace_arm}/base_link"/>
       <origin xyz="0.0 0 -${3*height/4}" rpy="0 ${pi/2} 0"/>
     </joint>
-    <!-- <gazebo reference="${namespace}/base_link"> -->
+    <!-- <gazebo reference="${namespace_arm}/base_link"> -->
     <gazebo reference="world_link_yaw">
       <selfCollide>false</selfCollide>
