Commit message: Redo Moveit config with Gazebo xacro
- Created a slightly modified xacro file for seabotix_base.xacro and seabotix_alpha.xacro
  which features added joints for moving and rotating the base.
- Reran the MoveIt! config on this modified xacro file

File: alpha_description/urdf/alpha_arm.xacro (robot description, xacro)
@@ -19,5 +19,5 @@
         <type>transmission_interface/SimpleTransmission</type>
         <joint name="${joint}">
-          <hardwareInterface>EffortJointInterface</hardwareInterface>
+          <hardwareInterface>hardware_interface/EffortJointInterface</hardwareInterface>
         </joint>
         <actuator name="${joint}_motor">

File: seabotix_alpha_description/urdf/seabotix_base_moveit.xacro (robot description, xacro)
@@ -39,7 +39,41 @@
   <xacro:property name="height" value="0.4572"/>
   <xacro:macro name="seabotix_base" params="namespace *gazebo inertial_reference_frame">
-    <!-- Create a dummy link to avoid :KDL does not support a root link with an inertia warning. -->
-    <!-- <link name="${namespace}/dummy_link"/>       -->
     <!-- base_link according to ROS conventions: x forward, z up -->
+    <link name="${namespace}/world_link_x">
+        <inertial>
+        <mass value="0" />
+        <origin xyz="0 0 0" rpy="0 0 0"/>
+        <inertia ixx="0" ixy="0" ixz="0"
+                iyy="0" iyz="0"
+                izz="0" />
+        </inertial>
+    </link>
+    <link name="${namespace}/world_link_y">
+        <inertial>
+        <mass value="0" />
+        <origin xyz="0 0 0" rpy="0 0 0"/>
+        <inertia ixx="0" ixy="0" ixz="0"
+                iyy="0" iyz="0"
+                izz="0" />
+        </inertial>
+    </link>
+    <link name="${namespace}/world_link_z">
+        <inertial>
+        <mass value="0" />
+        <origin xyz="0 0 0" rpy="0 0 0"/>
+        <inertia ixx="0" ixy="0" ixz="0"
+                iyy="0" iyz="0"
+                izz="0" />
+        </inertial>
+    </link>
+    <link name="${namespace}/world_link_yaw">
+        <inertial>
+        <mass value="0" />
+        <origin xyz="0 0 0" rpy="0 0 0"/>
+        <inertia ixx="0" ixy="0" ixz="0"
+                iyy="0" iyz="0"
+                izz="0" />
+        </inertial>
+    </link>
     <link name="${namespace}/base_link">
       <inertial>
@@ -64,8 +98,32 @@
       </collision>
     </link>
-    <!-- <joint name="${namespace}/dummy_to_base" type="fixed">
-      <parent link="${namespace}/dummy_link"/>
+    <joint name="x_displacement" type="prismatic">
+      <parent link="${namespace}/world_link_x"/>
+      <child link="${namespace}/world_link_y"/>
+      <origin rpy="0 0 0" xyz="0 0 0"/>
+      <axis xyz="1 0 0"/>
+      <limit effort="100" velocity="0.5" lower="-100" upper="100" /> <!-- Assume we are operating in 200x200x200m cube-->
+    </joint>
+    <joint name="y_displacement" type="prismatic">
+      <parent link="${namespace}/world_link_y"/>
+      <child link="${namespace}/world_link_z"/>
+      <origin rpy="0 0 0" xyz="0 0 0"/>
+      <axis xyz="0 1 0"/>
+      <limit effort="100" velocity="0.5" lower="-100" upper="100" /> <!-- Assume we are operating in 200x200x200m cube-->
+    </joint>
+    <joint name="z_displacement" type="prismatic">
+      <parent link="${namespace}/world_link_z"/>
+      <child link="${namespace}/world_link_yaw"/>
+      <origin rpy="0 0 0" xyz="0 0 0"/>
+      <axis xyz="0 0 1"/>
+      <limit effort="100" velocity="0.5" lower="-100" upper="100" /> <!-- Assume we are operating in 200x200x200m cube-->
+    </joint>
+    <joint name="yaw_displacement" type="continuous">
+      <parent link="${namespace}/world_link_yaw"/>
       <child link="${namespace}/base_link"/>
-    </joint> -->
+      <origin rpy="0 0 0" xyz="0 0 0"/>
+      <axis xyz="0 0 1"/>
+      <limit effort="100" velocity="${pi/10}"/> <!-- Assume we have no limit on yaw-->
+    </joint>
     <!-- Set up hydrodynamic plugin given as input parameter -->
     <xacro:insert_block name="gazebo"/>
